File: project/ch552-daplink/ch552-daplink.kicad_sch (KiCad schematic)
At the start: 16 parts, among them J1 USB_C_Receptacle_USB2.0_16P, J2 Conn_01x06_Pin, J3 BOOT, U1 CH552E

Commit message: 2025/07/17/20:12
Parts:
- J3: now not fitted
Changed lines of the file:
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@@
 		(in_bom yes)
 		(on_board yes)
-		(dnp no)
+		(dnp yes)
 		(fields_autoplaced yes)
 		(property "Reference" "J3"

Commit message: 2025/07/20/17:06
Parts:
- removed J2: Conn_01x06_Pin, Connector_Wuerth:Wuerth_WR-WTB_64800611622_1x06_P1.50mm_Vertical, symbol Connector:Conn_01x06_Pin
- added TP1, TP2, TP3, TP4, TP5, TP6: TestPoint, Connector_Wire:SolderWirePad_1x01_SMD_1x2mm, symbol Connector:TestPoint
Connections:
- net +3.3V: now also TP5.1
- net +5V: now also TP6.1
- net GND: now also TP1.1
- net at R7.2: now also TP3.1
- net at R8.2: now also TP2.1
- net at R6.1: now also TP4.1
