File: project/ch552-daplink/ch552-daplink_vcut.kicad_pcb (KiCad board)
At the start: 2 copper layers, 88 x 92 mm, 672 parts, among them J1 USB_C_Receptacle_USB2.0_16P, J3 BOOT, U1 CH552E

Commit message: 2025/07/21/19:49
Other:
- board text added: "←V-Cut"
Changed lines of the file:
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@@
+		)
+	)
+	(gr_text "←V-Cut"
+		(at 123.5 179.5 270)
+		(layer "Edge.Cuts")
+		(effects
+			(font
+				(size 1.5 1.5)
+				(thickness 0.3)
+				(bold yes)
+			)
+			(justify left)
+		)
+	)
+	(gr_text "←V-Cut"
+		(at 145.5 168 0)
+		(layer "Edge.Cuts")
+		(effects
+			(font
+				(size 1.5 1.5)
+				(thickness 0.3)
+				(bold yes)
+			)
+			(justify left)
+		)
+	)
+	(gr_text "←V-Cut"
+		(at 145.5 110.5 0)
+		(layer "Edge.Cuts")
+		(effects
+			(font
+				(size 1.5 1.5)
+				(thickness 0.3)
+				(bold yes)
+			)
+			(justify left)
+		)
+	)
+	(gr_text "←V-Cut"
+		(at 145.5 99 0)
+		(layer "Edge.Cuts")
+		(effects
+			(font
+				(size 1.5 1.5)
+				(thickness 0.3)
+				(bold yes)
+			)
+			(justify left)
+		)
+	)
+	(gr_text "←V-Cut"
+		(at 145.5 122 0)
+		(layer "Edge.Cuts")
+		(effects
+			(font
+				(size 1.5 1.5)
+				(thickness 0.3)
+				(bold yes)
+			)
+			(justify left)
+		)
+	)
+	(gr_text "←V-Cut"
+		(at 101.5 179.5 270)
+		(layer "Edge.Cuts")
+		(effects
+			(font
+				(size 1.5 1.5)
+				(thickness 0.3)
+				(bold yes)
+			)
+			(justify left)
+		)
+	)
+	(gr_text "←V-Cut"
+		(at 145.5 145 0)
+		(layer "Edge.Cuts")
+		(effects
+			(font
+				(size 1.5 1.5)
+				(thickness 0.3)
+				(bold yes)
+			)
+			(justify left)
+		)
+	)
+	(gr_text "←V-Cut"
+		(at 79.5 179.5 270)
+		(layer "Edge.Cuts")
+		(effects
+			(font
+				(size 1.5 1.5)
+				(thickness 0.3)
+				(bold yes)
+			)
+			(justify left)
+		)
+	)
+	(gr_text "←V-Cut"
+		(at 145.5 156.5 0)
+		(layer "Edge.Cuts")
+		(effects
+			(font
+				(size 1.5 1.5)
+				(thickness 0.3)
+				(bold yes)
+			)
+			(justify left)
+		)
+	)
+	(gr_text "←V-Cut"
+		(at 145.5 133.5 0)
+		(layer "Edge.Cuts")
+		(effects
+			(font
+				(size 1.5 1.5)
+				(thickness 0.3)
+				(bold yes)
+			)
+			(justify left)
 		)
 	)
