File: project/ch552-daplink/ch552-daplink.kicad_pcb (KiCad board)
At the start: 2 copper layers, 23 x 11.5 mm, 16 parts, among them J1 USB_C_Receptacle_USB2.0_16P, J2 Conn_01x06_Pin, J3 BOOT, U1 CH552E

Commit message: 2025/07/20/17:06
Parts:
- removed J2: Conn_01x06_Pin, Connector_Wuerth:Wuerth_WR-WTB_64800611622_1x06_P1.50mm_Vertical
- added TP1: TestPoint, Connector_Wire:SolderWirePad_1x01_SMD_1x2mm, F.Cu at (74.0, 84.0)
- added TP2: TestPoint, Connector_Wire:SolderWirePad_1x01_SMD_1x2mm, F.Cu at (74.0, 85.5)
- added TP3: TestPoint, Connector_Wire:SolderWirePad_1x01_SMD_1x2mm, F.Cu at (74.0, 87.0)
- added TP4: TestPoint, Connector_Wire:SolderWirePad_1x01_SMD_1x2mm, F.Cu at (74.0, 88.5)
- added TP5: TestPoint, Connector_Wire:SolderWirePad_1x01_SMD_1x2mm, F.Cu at (74.0, 90.0)
- added TP6: TestPoint, Connector_Wire:SolderWirePad_1x01_SMD_1x2mm, F.Cu at (74.0, 91.5)
Routing:
- net +3.3V: track 23.5 -> 22.0 mm
- net +5V: track 26.4 -> 25.4 mm
- net Net-(R8-Pad2): track 4.43 -> 3.70 mm
- net Net-(R7-Pad2): track 4.43 -> 3.70 mm
- net Net-(R6-Pad1): track 4.43 -> 3.70 mm
Other:
- board size 23 x 11.5 mm -> 22 x 11.5 mm
- board text added: "3.3V"
- board text added: "5V"
- board text added: "BOOT"
- board text added: "CH552-DAPLink v1.0.0 @netetra07"
- board text added: "GND"
- board text added: "RST"
- board text added: "SWCLK"
- board text added: "SWDIO"
- board text removed: "CH552-DAPLink @netetra07"
