File: project/ch334-usbhub/ch334-usbhub.kicad_pcb (KiCad board)
At the start: 2 copper layers, 95 x 30 mm, 32 parts, among them J1 USB_C_Receptacle_USB2.0_16P, J2 USB_A, J3 USB_A, J4 USB_A, J5 USB_A, U1 CH334R, U10 CH217, U2 USBLC6-2SC6, U3 USBLC6-2SC6, U4 CH217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

Commit message: 2025/07/27/13:56
Parts:
- added R7: 56kΩ, Resistor_SMD:R_0603_1608Metric, F.Cu at (104.0, 89.2)
- added U11: CH217, Package_TO_SOT_SMD:SOT-23-6, F.Cu at (102.9, 86.7)
Connections:
- J1 pad A4: +5V -> Net-(U11-VIN)
- J1 pad A9: +5V -> Net-(U11-VIN)
- J1 pad B4: +5V -> Net-(U11-VIN)
- J1 pad B9: +5V -> Net-(U11-VIN)
- U2 pad 5: +5V -> Net-(U11-VIN)
Routing:
- net Net-(U11-VIN): track 0.00 -> 16.3 mm, vias 0 -> 2
- net +5V: track 132.4 -> 116.4 mm, vias 7 -> 5
- net Net-(U11-ISET): track 0.00 -> 3.53 mm
- net GND: vias 145 -> 140
