File: project/ch334-usbhub/ch334-usbhub.kicad_sch (KiCad schematic)
At the start: 32 parts, among them J1 USB_C_Receptacle_USB2.0_16P, J2 USB_A, J3 USB_A, J4 USB_A, J5 USB_A, U1 CH334R, U10 CH217, U2 USBLC6-2SC6, U3 USBLC6-2SC6, U4 CH217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

Commit message: 2025/07/27/13:56
Parts:
- added R7: 56kΩ, Resistor_SMD:R_0603_1608Metric, symbol Device:R
- added U11: CH217, Package_TO_SOT_SMD:SOT-23-6, symbol CH21x:CH217K
Connections:
- net +5V: now also U11.1 (VOUT); no longer J1.A4 (VBUS), J1.A9 (VBUS), J1.B4 (VBUS), J1.B9 (VBUS), U2.5 (VBUS)
- net GND: now also R7.2, U11.2 (GND), U11.4 (EN#)
- new net: R7.1, U11.5 (ISET)
- new net: J1.A4 (VBUS), J1.A9 (VBUS), J1.B4 (VBUS), J1.B9 (VBUS), U11.6 (VIN), U2.5 (VBUS)
- no-connect marks 9 -> 10
Other:
- note added: "Q = CV C = 470 + 100 * 4 = 870uF Q = 870 * 5 = 4.35mC T = Q / I = 4.35mC / 1A = 4.35ms usbポートに刺して4.35msで使えるようになる"
- moved on the sheet: C1, J1, R1, R2, U2
