File: project/motor-driver/dc-v1/dc-v1.kicad_sch (KiCad schematic)
At the start: 6 parts, among them Q1 NMOS, Q2 NMOS

Commit message: 2025/09/22/19:15
Parts:
- removed Q1, Q2: NMOS, symbol Simulation_SPICE:NMOS
- added C1, C2: 1uF, Capacitor_SMD:C_0805_2012Metric, symbol Device:C
- added C10, C11, C12, C13, C6, C7, C8, C9: 0.1uF, Capacitor_SMD:C_0603_1608Metric, symbol Device:C
- added C3: 100uF, Capacitor_THT:CP_Radial_D8.0mm_P3.50mm, symbol Device:C_Polarized
- added C4: 47uF, Capacitor_THT:CP_Radial_D6.3mm_P2.50mm, symbol Device:C_Polarized
- added C5: 0.47uF, Capacitor_SMD:C_0603_1608Metric, symbol Device:C
- added D1, D2: 1N4148W, Diode_SMD:D_SOD-123, symbol Device:D_Schottky
- added D3, D4, D5: LED, LED_SMD:LED_0603_1608Metric, symbol Device:LED
- added H1, H2, H3, H4: MountingHole, MountingHole:MountingHole_3.2mm_M3, symbol Mechanical:MountingHole
- added J1: Power, Connector_AMASS:AMASS_XT30PW-M_1x02_P2.50mm_Horizontal, symbol Connector:Conn_01x02_Socket
- added J2: Motor, Connector_AMASS:AMASS_XT30PW-F_1x02_P2.50mm_Horizontal, symbol Connector:Conn_01x02_Socket
- added J3: Control, Connector_JST:JST_XH_S4B-XH-A_1x04_P2.50mm_Horizontal, symbol Connector:Conn_01x04_Pin
- added Q1, Q2, Q3, Q4: NMOS, Package_TO_SOT_SMD:TO-252-2, symbol Transistor_FET_Other:Q_NMOS_Depletion_GDS
- added R10, R13, R14, R6, R8, R9: 10kΩ, Resistor_SMD:R_0603_1608Metric, symbol Device:R
- added R11, R12: 1kΩ, Resistor_SMD:R_0603_1608Metric, symbol Device:R
- added R5, R7: 10Ω, Resistor_SMD:R_0603_1608Metric, symbol Device:R
- added U1, U2: IR2302, Package_SO:SOIC-8_3.9x4.9mm_P1.27mm, symbol Driver_FET:IR2302
- added U3: ADuM120N, Package_SO:SOIC-8_3.9x4.9mm_P1.27mm, symbol Isolator:ADuM120N
- added U4: L7805, Package_TO_SOT_SMD:TO-252-2, symbol Regulator_Linear:L7805
- added U5: 74AHC1G04, Package_TO_SOT_SMD:SOT-23-5, symbol 74xGxx:74AHC1G04
- added U6, U7: 74AHC1G08, Package_TO_SOT_SMD:SOT-23-5, symbol 74xGxx:74AHC1G08
- R1, R3: value R -> 10Ω; footprint (none) -> Resistor_SMD:R_0603_1608Metric
- R2, R4: value R -> 10kΩ; footprint (none) -> Resistor_SMD:R_0603_1608Metric
Connections:
- net at R3.1: now also U1.5 (LO)
- net at R3.2, R4.1: now also Q2.1 (G)
- net at R1.2, R2.1: now also Q1.1 (G)
- net MOTOR_A: now reaches R2.2
- net MOTOR_A: now also C1.2, J2.2 (Pin_2), Q1.3 (S), Q2.2 (D), R13.1, U1.6 (VS)
- net GND2: now reaches R4.2
- net GND2: now also C10.2, C11.2, C12.2, C13.1, C3.2, C4.2, C5.2, C6.2, C7.2, C8.2, J1.1 (Pin_1), Q2.3 (S), Q4.3 (S), R8.2, U1.4 (COM), U2.4 (COM), U3.5 (GND2), U4.2 (GND), U5.3 (GND), U6.3 (GND), U7.3 (GND)
- net at R1.1: now also U1.7 (HO)
- new net: C2.1, D2.1 (K), U2.8 (VB)
- new net: D5.2 (A), R14.1
- new net: Q3.1 (G), R5.2, R6.1
- new net: J3.3 (Pin_3), R9.1, U3.2 (VIA)
- new net: J3.2 (Pin_2), R10.1, U3.3 (VIB)
- new net: R12.1, U3.6 (VOB)
- new net: R11.1, U3.7 (VOA)
- new net: R7.1, U2.5 (LO)
- new net: R5.1, U2.7 (HO)
- new net: D3.1 (K), D4.2 (A), R13.2
- new net: U5.4, U6.2
- new net: Q4.1 (G), R7.2, R8.1
- new net: C1.1, D1.1 (K), U1.8 (VB)
- new net +12V: C3.1, C4.1, C5.1, C7.1, C8.1, D1.2 (A), D2.2 (A), J1.2 (Pin_2), Q1.2 (D), Q3.2 (D), U1.1 (VCC), U2.1 (VCC), U4.1 (IN)
- new net +5V: C10.1, C11.1, C12.1, C13.2, C6.1, R14.2, U3.8 (VDD2), U4.3 (OUT), U5.5 (VCC), U6.5 (VCC), U7.5 (VCC)
- new net DIR: R12.2, U5.2, U7.2
- new net GND: D5.1 (K)
- new net GND1: C9.2, J3.1 (Pin_1), R10.2, R9.2, U3.4 (GND1)
- new net IN_A: U1.2 (IN), U7.4
- new net IN_B: U2.2 (IN), U6.4
- new net MOTOR_B: C2.2, D3.2 (A), D4.1 (K), J2.1 (Pin_1), Q3.3 (S), Q4.2 (D), R6.2, U2.6 (VS)
- new net PWM: R11.2, U6.1, U7.1
- new net VCC: C9.1, J3.4 (Pin_4), U3.1 (VDD1)
- no-connect marks 0 -> 2
