File: project/motor-driver/dc-v1/dc-v1.kicad_pcb (KiCad board)
At the start: 2 copper layers, 61 x 43 mm, 50 parts, among them J1 Power, J2 Motor, J3 Control, Q1 NMOS, Q2 NMOS, Q3 NMOS, Q4 NMOS, U1 IR2302, U2 IR2302, U3 ADuM120N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

Commit message: 2025/10/04/15:59
Connections:
- D5 pad 1: GND -> GND2
Other:
- board text added: "v1.0.2"
- board text removed: "v1.0.0"
Changed lines of the file:
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@@
 	(net 29 "Net-(U5-Pad4)")
 	(net 30 "Net-(D5-A)")
-	(net 31 "GND")
 	(footprint "Diode_SMD:D_SOD-123"
 		(layer "F.Cu")
@@
 			(layers "F.Cu" "F.Mask" "F.Paste")
 			(roundrect_rratio 0.25)
-			(net 31 "GND")
+			(net 5 "GND2")
 			(pinfunction "K")
 			(pintype "passive")
@@
 		)
 	)
-	(gr_text "v1.0.0"
+	(gr_text "v1.0.2"
 		(at 149 97.25 90)
 		(layer "F.SilkS")
@@
 	)
 	(segment
+		(start 140 90)
+		(end 140 96.9)
+		(width 0.5)
+		(layer "F.Cu")
+		(net 18)
+	)
+	(segment
 		(start 140 96.9)
 		(end 140.35 97.25)
@@
 	)
 	(segment
-		(start 140 96)
-		(end 140 96.9)
+		(start 139.75 89.75)
+		(end 140 90)
 		(width 0.5)
 		(layer "F.Cu")
@@
 	)
 	(via
-		(at 140 96)
+		(at 139.75 89.75)
 		(size 0.6)
 		(drill 0.45)
@@
 	)
 	(segment
-		(start 126.75 80.345)
-		(end 126.75 87.75)
+		(start 139.75 89.75)
+		(end 138 88)
 		(width 0.5)
 		(layer "B.Cu")
@@
 	)
 	(segment
-		(start 138 88)
-		(end 140 90)
+		(start 126.75 87.75)
+		(end 126.75 80.345)
 		(width 0.5)
 		(layer "B.Cu")
@@
 	)
 	(segment
-		(start 126.75 87.75)
+		(start 138 88)
 		(end 127 88)
 		(width 0.5)
@@
 	)
 	(segment
-		(start 119.9525 73.5475)
-		(end 126.75 80.345)
+		(start 126.75 80.345)
+		(end 119.9525 73.5475)
 		(width 0.5)
 		(layer "B.Cu")
@@
 	(segment
 		(start 127 88)
-		(end 138 88)
-		(width 0.5)
-		(layer "B.Cu")
-		(net 18)
-	)
-	(segment
-		(start 140 90)
-		(end 140 96)
+		(end 126.75 87.75)
 		(width 0.5)
 		(layer "B.Cu")

Commit message: 2025/10/07/12:20
Routing:
- net GND2: vias 152 -> 161
Other:
- board text added: "v1.0.3"
- board text removed: "v1.0.2"
Changed lines of the file:
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@@
 	)
 	(gr_text "CW"
-		(at 134 104 0)
+		(at 137.5 102 0)
 		(layer "F.SilkS")
 		(effects
@@
 		)
 	)
-	(gr_text "v1.0.2"
+	(gr_text "v1.0.3"
 		(at 149 97.25 90)
 		(layer "F.SilkS")
@@
 	)
 	(gr_text "CCW"
-		(at 144 104 0)
+		(at 148.2 102 0)
 		(layer "F.SilkS")
 		(effects
@@
 	)
 	(via
+		(at 133 103)
+		(size 0.6)
+		(drill 0.45)
+		(layers "F.Cu" "B.Cu")
+		(free yes)
+		(net 5)
+	)
+	(via
 		(at 105.5 88.5)
 		(size 0.6)
@@
 	)
 	(via
+		(at 145 103)
+		(size 0.6)
+		(drill 0.45)
+		(layers "F.Cu" "B.Cu")
+		(free yes)
+		(net 5)
+	)
+	(via
 		(at 119.5 103)
 		(size 0.6)
@@
 	)
 	(via
+		(at 143.5 103)
+		(size 0.6)
+		(drill 0.45)
+		(layers "F.Cu" "B.Cu")
+		(free yes)
+		(net 5)
+	)
+	(via
+		(at 140.5 103)
+		(size 0.6)
+		(drill 0.45)
+		(layers "F.Cu" "B.Cu")
+		(free yes)
+		(net 5)
+	)
+	(via
 		(at 133 100)
 		(size 0.6)
@@
 	)
 	(via
+		(at 133 104.5)
+		(size 0.6)
+		(drill 0.45)
+		(layers "F.Cu" "B.Cu")
+		(free yes)
+		(net 5)
+	)
+	(via
 		(at 109.5 104.5)
 		(size 0.6)
@@
 	)
 	(via
+		(at 142 103)
+		(size 0.6)
+		(drill 0.45)
+		(layers "F.Cu" "B.Cu")
+		(free yes)
+		(net 5)
+	)
+	(via
 		(at 111.5 98.5)
 		(size 0.6)
@@
 	)
 	(via
+		(at 102 64)
+		(size 0.6)
+		(drill 0.45)
+		(layers "F.Cu" "B.Cu")
+		(free yes)
+		(net 5)
+	)
+	(via
 		(at 120 69.5)
 		(size 0.6)
@@
 	)
 	(via
+		(at 134.5 104.5)
+		(size 0.6)
+		(drill 0.45)
+		(layers "F.Cu" "B.Cu")
+		(free yes)
+		(net 5)
+	)
+	(via
 		(at 143.5 101.5)
 		(size 0.6)
@@
 	)
 	(via
+		(at 134.5 103)
+		(size 0.6)
+		(drill 0.45)
+		(layers "F.Cu" "B.Cu")
+		(free yes)
+		(net 5)
+	)
+	(via
 		(at 131.5 104.5)
 		(size 0.6)
@@
 	)
 	(segment
-		(start 140 90)
-		(end 140 96.9)
+		(start 139.5 89.5)
+		(end 140 90)
 		(width 0.5)
 		(layer "F.Cu")
@@
 	)
 	(segment
-		(start 140 96.9)
-		(end 140.35 97.25)
+		(start 119.905 73.5)
+		(end 119.905 72.275)
 		(width 0.5)
 		(layer "F.Cu")
@@
 	)
 	(segment
-		(start 119.905 73.5)
-		(end 119.905 72.275)
+		(start 119.9525 73.5475)
+		(end 119.905 73.5)
 		(width 0.5)
 		(layer "F.Cu")
@@
 	)
 	(segment
-		(start 119.9525 73.5475)
-		(end 119.905 73.5)
+		(start 140 96.9)
+		(end 140.35 97.25)
 		(width 0.5)
 		(layer "F.Cu")
@@
 	)
 	(segment
-		(start 139.75 89.75)
-		(end 140 90)
+		(start 140 90)
+		(end 140 96.9)
 		(width 0.5)
 		(layer "F.Cu")
@@
 	)
 	(via
-		(at 139.75 89.75)
+		(at 139.5 89.5)
 		(size 0.6)
 		(drill 0.45)
@@
 	)
 	(segment
-		(start 139.75 89.75)
+		(start 139.5 89.5)
 		(end 138 88)
 		(width 0.5)
@@
 	)
 	(segment
-		(start 126.75 87.75)
-		(end 126.75 80.345)
-		(width 0.5)
-		(layer "B.Cu")
-		(net 18)
-	)
-	(segment
 		(start 138 88)
 		(end 127 88)
@@
 		(width 0.5)
 		(layer "B.Cu")
+		(net 18)
+	)
+	(segment
+		(start 126.75 87.75)
+		(end 126.75 80.345)
+		(width 0.5)
+		(layer "B.Cu")
