File: project/motor-driver/dc-v2/dc-v2.kicad_pcb (KiCad board)
At the start: 2 copper layers, 79 parts, among them J1 Power, J2 Limit_A, J3 AMT102, J4 Limit_B, J5 CAN, J6 Motor, Q1 PMOS, Q2 NMOS, Q3 NMOS, Q4 NMOS, Q5 NMOS, U1 L7812, U10 INA180A1, U11 74AHC1G08, U12 IR2302, U13 74AHC1G08, U14 TC7W74, U2 L7805, U3 NJM12888, U4 STM32F303K8Tx, U5 MCP2562-E-SN, U6 74AHC1G08, U7 LM2904, U8 IR2302, U9 74AHC1G04

Commit message: 2025/10/14/08:57
Parts:
- removed C26, C29, C30, C32, C33, C34, C35: 0.1uF, Capacitor_SMD:C_0603_1608Metric
- removed C27, C31: 1uF, Capacitor_SMD:C_0805_2012Metric
- removed C28: C, Capacitor_SMD:C_0603_1608Metric
- removed Q5: NMOS, Package_TO_SOT_SMD:TO-252-2
- removed U11, U13: 74AHC1G08, Package_TO_SOT_SMD:SOT-23-5
- removed U12: IR2302, Package_SO:SOIC-8_3.9x4.9mm_P1.27mm
- removed U14: TC7W74, Package_SO:TSSOP-8_3x3mm_P0.65mm
- added C1: 0.1uF, Capacitor_SMD:C_0603_1608Metric, F.Cu at (33.5, 21.9)
- added C2: 0.1uF, Capacitor_SMD:C_0603_1608Metric, F.Cu at (33.5, 24.5)
- added C20: 0.1uF, Capacitor_SMD:C_0603_1608Metric, F.Cu at (37.5, 39.5)
- added D1: Blue, LED_SMD:LED_0603_1608Metric, F.Cu at (21.4, 71.2)
- added D6: Yellow, LED_SMD:LED_0603_1608Metric, F.Cu at (21.4, 81.5)
- added D7: 1N4148W, Diode_SMD:D_SOD-123, F.Cu at (76.6, 48.3)
- added D8: 1N4148W, Diode_SMD:D_SOD-123, F.Cu at (76.6, 51.7)
- added D9: 1N4148W, Diode_SMD:D_SOD-123, F.Cu at (76.6, 55.0)
- added H1: MountingHole, MountingHole:MountingHole_3.2mm_M3, F.Cu at (105.0, 54.0)
- added H2: MountingHole, MountingHole:MountingHole_3.2mm_M3, F.Cu at (174.0, 54.0)
- added H3: MountingHole, MountingHole:MountingHole_3.2mm_M3, F.Cu at (174.0, 104.0)
- added H4: MountingHole, MountingHole:MountingHole_3.2mm_M3, F.Cu at (105.0, 104.0)
- added J7: Debug, Connector_PinSocket_2.54mm:PinSocket_1x05_P2.54mm_Horizontal, F.Cu at (50.5, 63.4)
- added R1: 10kΩ, Resistor_SMD:R_0603_1608Metric, F.Cu at (41.5, 29.5)
- added R16: 10kΩ, Resistor_SMD:R_0603_1608Metric, F.Cu at (49.5, 21.9)
- added R21: 10Ω, Resistor_SMD:R_0603_1608Metric, F.Cu at (49.5, 34.5)
- added Y1: XT324 16MHz, Crystal:Crystal_SMD_3225-4Pin_3.2x2.5mm, F.Cu at (46.5, 78.2)
- C11, C12: value C -> 0.1uF
- C14: value 4.7uF -> 0.1uF
- C15: value 0.01uF -> 1uF; footprint Capacitor_SMD:C_0603_1608Metric -> Capacitor_SMD:C_0805_2012Metric
- C17, C19, C21: value 0.01uF -> 0.47uF
- C18, C24: value 0.1uF -> 0.47uF
- C22: value 0.1uF -> 1uF; footprint Capacitor_SMD:C_0603_1608Metric -> Capacitor_SMD:C_0805_2012Metric
- C3: value 0.47uF -> 100uF; footprint Capacitor_SMD:C_0603_1608Metric -> Capacitor_THT:CP_Radial_D8.0mm_P3.50mm
- C4: value 0.1uF -> 47uF; footprint Capacitor_SMD:C_0603_1608Metric -> Capacitor_THT:CP_Radial_D6.3mm_P2.50mm
- C5, C8: value 0.47uF -> 0.1uF
- C6, C7: value 0.1uF -> 10pF
- C9: value 0.1uF -> 4.7uF
- D2, D3, D5: value 1N4148W -> Yellow; footprint Diode_SMD:D_SOD-123 -> LED_SMD:LED_0603_1608Metric
- J2: value Limit_A -> Motor; footprint Connector_JST:JST_XH_S2B-XH-A_1x02_P2.50mm_Horizontal -> Connector_AMASS:AMASS_XT30PW-F_1x02_P2.50mm_Horizontal
- J3: value AMT102 -> CAN; footprint Connector_JST:JST_XH_S5B-XH-A_1x05_P2.50mm_Horizontal -> Connector_JST:JST_XA_S02B-XASK-1N-BN_1x02_P2.50mm_Horizontal
- J4: value Limit_B -> AMT102; footprint Connector_JST:JST_XH_S2B-XH-A_1x02_P2.50mm_Horizontal -> Connector_JST:JST_XH_S5B-XH-A_1x05_P2.50mm_Horizontal
- J5: value CAN -> Limit_A
- J6: value Motor -> Limit_B; footprint Connector_AMASS:AMASS_XT30PW-F_1x02_P2.50mm_Horizontal -> Connector_JST:JST_XH_S2B-XH-A_1x02_P2.50mm_Horizontal
- Q1: value PMOS -> NMOS
- R11, R12: value 10Ω -> 1kΩ
- R13: value R -> 10Ω
- R14: value 10kΩ -> 10Ω
- R19: value 10Ω -> 10kΩ
- R7: value 10kΩ -> 1kΩ
- U1: value L7812 -> 74AHC1G04; footprint Package_TO_SOT_SMD:TO-252-2 -> Package_TO_SOT_SMD:SOT-23-5
- U10: value INA180A1 -> MCP2562-E-SN; footprint Package_TO_SOT_SMD:SOT-23-5 -> Package_SO:SOIC-8_3.9x4.9mm_P1.27mm
- U2: value L7805 -> 74AHC1G08; footprint Package_TO_SOT_SMD:TO-252-2 -> Package_TO_SOT_SMD:SOT-23-5
- U3: value NJM12888 -> STM32F303K8Tx; footprint Package_TO_SOT_SMD:SOT-23-5 -> Package_QFP:LQFP-32_7x7mm_P0.8mm
- U4: value STM32F303K8Tx -> 74AHC1G08; footprint Package_QFP:LQFP-32_7x7mm_P0.8mm -> Package_TO_SOT_SMD:SOT-23-5
- U5: value MCP2562-E-SN -> IR2302
- U6: value 74AHC1G08 -> NJM12888
- U7: value LM2904 -> L7812; footprint Package_SO:SOIC-8_5.3x6.2mm_P1.27mm -> Package_TO_SOT_SMD:TO-252-2
- U9: value 74AHC1G04 -> L7805; footprint Package_TO_SOT_SMD:SOT-23-5 -> Package_TO_SOT_SMD:TO-252-2
- moved Q3 144.8 mm to (156.0, 98.3), turned to 180 degrees
- moved Q2 141.0 mm to (156.0, 81.3), turned to 180 degrees
- moved J6 130.9 mm to (166.2, 60.4), turned to 180 degrees
- moved Q4 128.6 mm to (142.0, 98.3), turned to 180 degrees
- moved J2 126.6 mm to (169.0, 90.0), turned to -90 degrees
- moved U7 84.9 mm to (107.0, 80.9), turned to 180 degrees
- moved J5 84.4 mm to (156.2, 60.4), turned to 180 degrees
- moved J4 83.7 mm to (146.0, 60.4), turned to 180 degrees
- moved Q1 78.4 mm to (142.0, 81.3), turned to 180 degrees
- moved U10 74.5 mm to (120.5, 63.0), turned to 180 degrees
- moved C5 66.9 mm to (33.5, 27.0)
- moved C6 66.9 mm to (33.5, 29.5)
- moved C7 66.9 mm to (33.5, 32.0)
- moved C8 66.9 mm to (33.5, 34.5)
- moved U9 66.2 mm to (107.0, 72.7), turned to 180 degrees
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Connections:
- C10 pad 1: LIMIT_A -> +3.3V
- C11 pad 1: GND -> +12V
- C11 pad 2: OSC_IN -> GND
- C12 pad 1: GND -> +3.3V
- C12 pad 2: OSC_OUT -> GND
- C13 pad 1: LIMIT_B -> +3.3V
- C15 pad 1: ENC_X -> Net-(D4-K)
- C15 pad 2: GND -> MOTOR_A
- C16 pad 1: +3.3V -> +5V
- C17 pad 1: ENC_A -> +BATT
- C19 pad 1: ENC_B -> +12V
- C21 pad 1: Net-(U4-VDDA) -> +BATT
- C22 pad 1: GND -> Net-(D8-K)
- C22 pad 2: +3.3V -> MOTOR_B
- C24 pad 1: +3.3V -> +5V
- C4 pad 1: +12V -> +BATT
- C5 pad 1: +BATT -> LIMIT_B
- C6 pad 1: +5V -> GND
- C6 pad 2: GND -> OSC_IN
- C7 pad 1: +5V -> GND
- C7 pad 2: GND -> OSC_OUT
- C9 pad 1: NRST -> +3.3V
- D2 pad 1: +BATT -> GND
- D2 pad 2: +12V -> Net-(D2-A)
- D3 pad 1: +BATT -> GND
- D3 pad 2: +5V -> Net-(D3-A)
- D5 pad 1: Net-(D5-K) -> MOTOR_A
- D5 pad 2: +12V -> Net-(D5-A)
- J1 pad 2: Net-(J1-Pin_2) -> +BATT
- J2 pad 1: GND -> MOTOR_B
- J2 pad 2: LIMIT_A -> MOTOR_A
- J3 pad 1: GND -> CAN-
- J3 pad 2: Net-(J3-Pin_2) -> CAN+
- J4 pad 2: LIMIT_B -> ENC_X
- J5 pad 1: CAN- -> GND
- J5 pad 2: CAN+ -> LIMIT_A
- J6 pad 1: MOTOR_B -> GND
- J6 pad 2: MOTOR_A -> LIMIT_B
- Q1 pad 1: Net-(J1-Pin_2) -> Net-(Q1-G)
- Q1 pad 2: Net-(D1-A) -> +BATT
- Q1 pad 3: +BATT -> MOTOR_A
- Q2 pad 2: +BATT -> MOTOR_A
- Q2 pad 3: MOTOR_A -> GND
- Q3 pad 2: MOTOR_A -> +BATT
- Q3 pad 3: Net-(Q3-S) -> MOTOR_B
- Q4 pad 2: +BATT -> MOTOR_B
- Q4 pad 3: MOTOR_B -> GND
- R10 pad 1: Net-(J3-Pin_2) -> +3.3V
- R10 pad 2: ENC_X -> Net-(D1-A)
- R11 pad 1: Net-(U8-HO) -> CAN_TX_IND
- R11 pad 2: Net-(Q2-G) -> Net-(D2-A)
- R12 pad 1: Net-(U8-LO) -> CAN_RX_IND
- R12 pad 2: Net-(Q3-G) -> Net-(D3-A)
- R13 pad 1: Net-(U7A-+) -> Net-(U5-HO)
- R13 pad 2: Net-(R13-Pad2) -> Net-(Q1-G)
- R14 pad 1: Net-(Q2-G) -> Net-(U5-LO)
- R14 pad 2: MOTOR_A -> Net-(Q2-G)
- R15 pad 1: Net-(Q3-G) -> MOTOR_B
- R15 pad 2: Net-(Q3-S) -> Net-(D5-A)
- R17 pad 1: Net-(Q4-G) -> Net-(Q2-G)
- R17 pad 2: MOTOR_B -> GND
- R18 pad 1: Net-(Q5-G) -> Net-(Q3-G)
- R18 pad 2: Net-(Q3-S) -> MOTOR_B
- R19 pad 1: Net-(U12-HO) -> Net-(Q4-G)
- R19 pad 2: Net-(Q4-G) -> GND
- R2 pad 1: +5V -> ENC_X
- R2 pad 2: LIMIT_A -> GND
- R20 pad 1: Net-(U12-LO) -> Net-(U8-HO)
- R20 pad 2: Net-(Q5-G) -> Net-(Q3-G)
- R3 pad 1: BOOT0 -> ENC_A
- R4 pad 1: Net-(J3-Pin_2) -> GND
- R4 pad 2: GND -> BOOT0
- R5 pad 1: +5V -> ENC_B
- R5 pad 2: LIMIT_B -> GND
- R6 pad 1: Net-(J3-Pin_3) -> +5V
- R6 pad 2: GND -> LIMIT_B
- R7 pad 1: Net-(J3-Pin_5) -> Net-(J7-Pin_4)
- R7 pad 2: GND -> NRST
- R8 pad 1: Net-(J3-Pin_5) -> Net-(J7-Pin_3)
- R8 pad 2: ENC_B -> SWDIO
- R9 pad 1: Net-(J3-Pin_3) -> Net-(J7-Pin_2)
- R9 pad 2: ENC_A -> SWCLK
- U1 pad 1: +BATT -> (no net)
- U1 pad 2: GND -> DIR
- U1 pad 3: +12V -> GND
- U10 pad 1: Net-(R13-Pad2) -> CAN_TX
- U10 pad 3: Net-(U10-+) -> +5V
- U10 pad 4: Net-(U10--) -> CAN_RX
- U10 pad 5: +5V -> +3.3V
- U2 pad 1: +BATT -> PWM
- U2 pad 2: GND -> Net-(U1-Pad4)
- U2 pad 3: +5V -> GND
- U3 pad 1: +5V -> +3.3V
- U3 pad 2: GND -> OSC_IN
- U3 pad 3: +5V -> OSC_OUT
- U3 pad 4: unconnected-(U3-Cs-Pad4) -> NRST
- U4 pad 1: +3.3V -> PWM
- U4 pad 2: OSC_IN -> DIR
- U4 pad 3: OSC_OUT -> GND
- U4 pad 4: NRST -> IN_B
- U4 pad 5: Net-(U4-VDDA) -> +3.3V
- U5 pad 1: CAN_TX -> +12V
- U5 pad 2: GND -> IN_A
- U5 pad 3: +5V -> unconnected-(U5-~{SD}-Pad3)
- U5 pad 4: CAN_RX -> GND
- U5 pad 5: +3.3V -> Net-(U5-LO)
- U5 pad 6: CAN- -> MOTOR_A
- U5 pad 7: CAN+ -> Net-(U5-HO)
- U5 pad 8: GND -> Net-(D4-K)
- U6 pad 1: PWM_SRC -> +5V
- U6 pad 2: PWM_ENABLE -> GND
- U6 pad 3: GND -> +5V
- U6 pad 4: PWM -> unconnected-(U6-Cs-Pad4)
- U7 pad 1: I_SENSE -> +BATT
- U7 pad 2: I_SENSE -> GND
- U7 pad 3: Net-(U7A-+) -> +12V
- U8 pad 2: IN_A -> IN_B
- U8 pad 6: MOTOR_A -> MOTOR_B
- U8 pad 8: Net-(D4-K) -> Net-(D8-K)
- U9 pad 1: (no net) -> +BATT
- U9 pad 2: DIR -> GND
- U9 pad 3: GND -> +5V
