File: project/motor-driver/dc-v2/mcu.kicad_sch (KiCad schematic)
At the start: 34 parts, among them J2 Limit_A, J3 AMT102, J4 Limit_B, J5 CAN, SW1 Reset, SW2 Boot, U4 STM32F303K8Tx, U5 MCP2562-E-SN, Y1 8MHz

Commit message: 2025/10/14/08:57
Parts:
- removed C10, C13, C16, C18, C22, C23, C9: 0.1uF, Capacitor_SMD:C_0603_1608Metric, symbol Device:C
- removed C11, C12: C, Capacitor_SMD:C_0603_1608Metric, symbol Device:C
- removed C14: 4.7uF, Capacitor_SMD:C_0603_1608Metric, symbol Device:C
- removed C15, C17, C19, C21: 0.01uF, Capacitor_SMD:C_0603_1608Metric, symbol Device:C
- removed C20: 1uF, symbol Device:C
- removed FB1: FerriteBead_Small, symbol Device:FerriteBead_Small
- removed J2: Limit_A, Connector_JST:JST_XH_S2B-XH-A_1x02_P2.50mm_Horizontal, symbol Connector:Conn_01x02_Socket
- removed J3: AMT102, Connector_JST:JST_XH_S5B-XH-A_1x05_P2.50mm_Horizontal, symbol Connector:Conn_01x05_Socket
- removed J4: Limit_B, Connector_JST:JST_XH_S2B-XH-A_1x02_P2.50mm_Horizontal, symbol Connector:Conn_01x02_Socket
- removed J5: CAN, Connector_JST:JST_XH_S2B-XH-A_1x02_P2.50mm_Horizontal, symbol Connector:Conn_01x02_Socket
- removed R10, R8, R9: 1kΩ, Resistor_SMD:R_0603_1608Metric, symbol Device:R
- removed R2, R3, R4, R5, R6, R7: 10kΩ, Resistor_SMD:R_0603_1608Metric, symbol Device:R
- removed SW1: Reset, symbol Switch:SW_Push
- removed SW2: Boot, symbol Switch:SW_Push
- removed U4: STM32F303K8Tx, Package_QFP:LQFP-32_7x7mm_P0.8mm, symbol MCU_ST_STM32F3:STM32F303K8Tx
- removed U5: MCP2562-E-SN, Package_SO:SOIC-8_3.9x4.9mm_P1.27mm, symbol Interface_CAN_LIN:MCP2562-E-SN
- removed Y1: 8MHz, symbol Device:Crystal_GND23
Connections:
- no-connect marks 19 -> 0
