File: project/motor-driver/dc-v2/motor-drive.kicad_sch (KiCad schematic)
At the start: 38 parts, among them J6 Motor, Q2 NMOS, Q3 NMOS, Q4 NMOS, Q5 NMOS, U10 INA180A1, U11 74AHC1G08, U12 IR2302, U13 74AHC1G08, U14 TC7W74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

Commit message: 2025/10/14/08:57
Parts:
- removed C24, C25, C26, C29, C30, C32, C33, C34, C35: 0.1uF, Capacitor_SMD:C_0603_1608Metric, symbol Device:C
- removed C27, C31: 1uF, Capacitor_SMD:C_0805_2012Metric, symbol Device:C
- removed C28: C, Capacitor_SMD:C_0603_1608Metric, symbol Device:C
- removed D4, D5: 1N4148W, Diode_SMD:D_SOD-123, symbol Device:D_Schottky
- removed J6: Motor, Connector_AMASS:AMASS_XT30PW-F_1x02_P2.50mm_Horizontal, symbol Connector:Conn_01x02_Socket
- removed Q2, Q3, Q4, Q5: NMOS, Package_TO_SOT_SMD:TO-252-2, symbol Transistor_FET_Other:Q_NMOS_Depletion_GDS
- removed R11, R12, R19, R20: 10Ω, Resistor_SMD:R_0603_1608Metric, symbol Device:R
- removed R13: R, Resistor_SMD:R_0603_1608Metric, symbol Device:R
- removed R14, R15, R17, R18: 10kΩ, Resistor_SMD:R_0603_1608Metric, symbol Device:R
- removed R16: 5mΩ, symbol Device:R_Shunt
- removed U10: INA180A1, Package_TO_SOT_SMD:SOT-23-5, symbol Amplifier_Current:INA180A1
- removed U11, U13, U6: 74AHC1G08, Package_TO_SOT_SMD:SOT-23-5, symbol 74xGxx:74AHC1G08
- removed U12, U8: IR2302, Package_SO:SOIC-8_3.9x4.9mm_P1.27mm, symbol Driver_FET:IR2302
- removed U14: TC7W74, Package_SO:TSSOP-8_3x3mm_P0.65mm, symbol TOSHIBA_LogicGate:TC7W74
- removed U7: LM2904, Package_SO:SOIC-8_5.3x6.2mm_P1.27mm, symbol Amplifier_Operational:LM2904
- removed U9: 74AHC1G04, Package_TO_SOT_SMD:SOT-23-5, symbol 74xGxx:74AHC1G04
Connections:
- no-connect marks 3 -> 0
Other:
- note removed: "過電流でLow"
