File: project/research/ch559-dev-board/ch559-dev-board.kicad_pcb (KiCad board)
At the start: 2 copper layers, 0 parts

Commit message: 2025/11/09/00:50
Parts:
- added C1: 22uF, Capacitor_THT:CP_Radial_D6.3mm_P2.50mm, F.Cu at (200.0, 70.0)
- added C2: 22uF, Capacitor_THT:CP_Radial_D6.3mm_P2.50mm, F.Cu at (200.0, 105.0)
- added C3: 0.1uF, Capacitor_THT:C_Disc_D5.1mm_W3.2mm_P5.00mm, F.Cu at (153.0, 68.0)
- added C4: 4.7uF, Capacitor_THT:C_Disc_D5.1mm_W3.2mm_P5.00mm, F.Cu at (143.5, 68.0)
- added C5: 10uF, Capacitor_THT:C_Disc_D5.1mm_W3.2mm_P5.00mm, F.Cu at (160.8, 65.0)
- added C6: 22uF, Capacitor_THT:C_Disc_D5.1mm_W3.2mm_P5.00mm, F.Cu at (160.8, 53.0)
- added C7: 1uF, Capacitor_THT:C_Disc_D5.1mm_W3.2mm_P5.00mm, F.Cu at (153.0, 64.0)
- added D1: LED, LED_THT:LED_D5.0mm, F.Cu at (174.0, 39.5)
- added D2: LED, LED_THT:LED_D5.0mm, F.Cu at (181.0, 39.5)
- added D3: LED, LED_THT:LED_D5.0mm, F.Cu at (188.0, 39.5)
- added D4: D_Schottky, Diode_THT:D_A-405_P10.16mm_Horizontal, F.Cu at (157.8, 64.1)
- added J1: USB_C_Receptacle_USB2.0_16P, breakout_board:usbc-dip, F.Cu at (130.0, 55.0)
- added J2: USB_A, breakout_board:usb-dip, F.Cu at (192.4, 92.5)
- added J3: USB_A, breakout_board:usb-dip, F.Cu at (192.4, 57.4)
- added J4: UART, Connector_PinHeader_2.54mm:PinHeader_1x04_P2.54mm_Vertical, F.Cu at (186.0, 65.5)
- added J5: LED, Connector_PinHeader_2.54mm:PinHeader_1x02_P2.54mm_Vertical, F.Cu at (175.0, 63.0)
- added J6: UART_SIG, Connector_PinHeader_2.54mm:PinHeader_1x02_P2.54mm_Vertical, F.Cu at (179.0, 60.5)
- added J7: Conn_01x24_Pin, Connector_PinSocket_2.54mm:PinSocket_1x24_P2.54mm_Vertical, F.Cu at (130.0, 107.5)
- added J8: Conn_01x24_Pin, Connector_PinSocket_2.54mm:PinSocket_1x24_P2.54mm_Vertical, F.Cu at (188.4, 72.5)
- added R1: 5.1kΩ, Resistor_THT:R_Axial_DIN0207_L6.3mm_D2.5mm_P10.16mm_Horizontal, F.Cu at (129.8, 42.5)
- added R2: 5.1kΩ, Resistor_THT:R_Axial_DIN0207_L6.3mm_D2.5mm_P10.16mm_Horizontal, F.Cu at (129.8, 38.5)
- added R3: 1kΩ, Resistor_THT:R_Axial_DIN0207_L6.3mm_D2.5mm_P10.16mm_Horizontal, F.Cu at (171.9, 47.0)
- added R4: 1kΩ, Resistor_THT:R_Axial_DIN0207_L6.3mm_D2.5mm_P10.16mm_Horizontal, F.Cu at (171.9, 52.0)
- added R5: 1kΩ, Resistor_THT:R_Axial_DIN0207_L6.3mm_D2.5mm_P10.16mm_Horizontal, F.Cu at (171.9, 55.0)
- added R6: 1kΩ, Resistor_THT:R_Axial_DIN0207_L6.3mm_D2.5mm_P10.16mm_Horizontal, F.Cu at (146.0, 48.2)
- added R7: 1kΩ, Resistor_THT:R_Axial_DIN0207_L6.3mm_D2.5mm_P10.16mm_Horizontal, F.Cu at (159.0, 48.1)
- added SW1: RESET, Button_Switch_THT:SW_PUSH_6mm, F.Cu at (149.8, 46.2)
- added SW2: BOOT, Button_Switch_THT:SW_PUSH_6mm, F.Cu at (162.8, 46.2)
- added SW3: SW_Slide_DPDT, Button_Switch_THT:SW_CK_JS202011CQN_DPDT_Straight, F.Cu at (146.0, 60.3)
- added U1: CH559L, breakout:qfp48-dip, F.Cu at (130.0, 90.0)
- added U2: AZ1117CH2-3.3, Package_TO_SOT_SMD:SOT-223-3_TabPin2, B.Cu at (164.0, 59.0)
Routing:
- net GND: track 0.00 -> 397.6 mm, vias 0 -> 2
- net VBUS: track 0.00 -> 161.1 mm, vias 0 -> 6
- net D0+: track 0.00 -> 81.2 mm
- net D0-: track 0.00 -> 80.6 mm
- net +3.3V: track 0.00 -> 70.6 mm
- net D1-: track 0.00 -> 60.7 mm
- net D1+: track 0.00 -> 58.4 mm
- net BOOT: track 0.00 -> 24.1 mm
- net RST: track 0.00 -> 19.7 mm
- net Net-(D3-A): track 0.00 -> 15.5 mm
- net Net-(D2-A): track 0.00 -> 14.0 mm
- net 42: track 0.00 -> 13.8 mm
- net Net-(J1-CC2): track 0.00 -> 13.6 mm
- net Net-(J1-CC1): track 0.00 -> 12.1 mm
- net Net-(D1-A): track 0.00 -> 10.2 mm
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Other:
- board outline added: 92 x 75 mm
