File: project/research/ch559-dev-board/ch559-dev-board.kicad_sch (KiCad schematic)
At the start: 0 parts

Commit message: 2025/11/09/00:50
Parts:
- added C1, C2: 22uF, Capacitor_THT:CP_Radial_D6.3mm_P2.50mm, symbol Device:C_Polarized
- added C3: 0.1uF, Capacitor_THT:C_Disc_D5.1mm_W3.2mm_P5.00mm, symbol Device:C
- added C4: 4.7uF, Capacitor_THT:C_Disc_D5.1mm_W3.2mm_P5.00mm, symbol Device:C
- added C5: 10uF, Capacitor_THT:C_Disc_D5.1mm_W3.2mm_P5.00mm, symbol Device:C
- added C6: 22uF, Capacitor_THT:C_Disc_D5.1mm_W3.2mm_P5.00mm, symbol Device:C
- added C7: 1uF, Capacitor_THT:C_Disc_D5.1mm_W3.2mm_P5.00mm, symbol Device:C
- added D1, D2, D3: LED, LED_THT:LED_D5.0mm, symbol Device:LED
- added D4: D_Schottky, Diode_THT:D_A-405_P10.16mm_Horizontal, symbol Device:D_Schottky
- added J1: USB_C_Receptacle_USB2.0_16P, breakout_board:usbc-dip, symbol Connector:USB_C_Receptacle_USB2.0_16P
- added J2, J3: USB_A, breakout_board:usb-dip, symbol Connector:USB_A
- added J4: UART, Connector_PinHeader_2.54mm:PinHeader_1x04_P2.54mm_Vertical, symbol Connector:Conn_01x04_Pin
- added J5: LED, Connector_PinHeader_2.54mm:PinHeader_1x02_P2.54mm_Vertical, symbol Connector:Conn_01x02_Pin
- added J6: UART_SIG, Connector_PinHeader_2.54mm:PinHeader_1x02_P2.54mm_Vertical, symbol Connector:Conn_01x02_Pin
- added J7, J8: Conn_01x24_Pin, Connector_PinSocket_2.54mm:PinSocket_1x24_P2.54mm_Vertical, symbol Connector:Conn_01x24_Pin
- added R1, R2: 5.1kΩ, Resistor_THT:R_Axial_DIN0207_L6.3mm_D2.5mm_P10.16mm_Horizontal, symbol Device:R
- added R3, R4, R5, R6, R7: 1kΩ, Resistor_THT:R_Axial_DIN0207_L6.3mm_D2.5mm_P10.16mm_Horizontal, symbol Device:R
- added SW1: RESET, Button_Switch_THT:SW_PUSH_6mm, symbol Switch:SW_Push
- added SW2: BOOT, Button_Switch_THT:SW_PUSH_6mm, symbol Switch:SW_Push
- added SW3: SW_Slide_DPDT, Button_Switch_THT:SW_CK_JS202011CQN_DPDT_Straight, symbol Switch:SW_Slide_DPDT
- added U1: CH559L, breakout:qfp48-dip, symbol CH55x:CH559L
- added U2: AZ1117CH2-3.3, Package_TO_SOT_SMD:SOT-223-3_TabPin2, symbol Regulator_Linear:AZ1117CH2-3.3
Connections:
- new net: J1.A5 (CC1), R1.1
- new net: J1.B5 (CC2), R2.1
- new net: J5.2 (Pin_2), R4.1
- new net: D2.2 (A), R4.2
- new net: D1.2 (A), R3.2
- new net: J4.3 (Pin_3), J6.1 (Pin_1)
- new net: J4.2 (Pin_2), J6.2 (Pin_2)
- new net: D3.2 (A), R5.2
- new net: J5.1 (Pin_1), R5.1
- new net +3.3V: C6.1, D4.2 (A), J4.1 (Pin_1), R3.1, R7.1, SW1.2, U2.3 (OUT)
- new net 1: J7.1 (Pin_1), U1.1 (P1.6)
- new net 10: J7.10 (Pin_10), U1.10 (P3.4)
- new net 11: J7.11 (Pin_11), U1.11 (P3.5)
- new net 12: J7.12 (Pin_12), U1.12 (P3.6)
- new net 13: J7.13 (Pin_13), U1.13 (P3.7)
- new net 14: J7.14 (Pin_14), U1.14 (P4.3)
- new net 15: J7.15 (Pin_15), U1.15 (P4.2)
- new net 17: J7.17 (Pin_17), U1.17 (P4.7)
- new net 19: J7.19 (Pin_19), U1.19 (P4.1)
- new net 2: J7.2 (Pin_2), U1.2 (P1.7)
- new net 20: J7.20 (Pin_20), U1.20 (P4.0)
- new net 21: J7.21 (Pin_21), U1.21 (P2.0)
- new net 22: J7.22 (Pin_22), U1.22 (P2.1)
- new net 23: J7.23 (Pin_23), U1.23 (P2.2)
- new net 24: J7.24 (Pin_24), U1.24 (P2.3)
- new net 25: J8.1 (Pin_1), U1.25 (P2.4)
- new net 26: J8.2 (Pin_2), U1.26 (P2.5)
- new net 27: J8.3 (Pin_3), U1.27 (P2.6)
- new net 28: J8.4 (Pin_4), U1.28 (P2.7)
- new net 33: J8.9 (Pin_9), U1.33 (P0.7)
- new net 34: J8.10 (Pin_10), U1.34 (P0.6)
- new net 35: J8.11 (Pin_11), U1.35 (P0.5)
- new net 36: J8.12 (Pin_12), U1.36 (P0.4)
- new net 37: J8.13 (Pin_13), U1.37 (P0.3)
- new net 38: J8.14 (Pin_14), U1.38 (P0.2)
- new net 39: J8.15 (Pin_15), U1.39 (P0.1)
- new net 4: J7.4 (Pin_4), U1.4 (P3.0)
- new net 40: J8.16 (Pin_16), U1.40 (P0.0)
- new net 42: C4.1, J8.18 (Pin_18), U1.42 (VDD33)
- new net 43: J8.19 (Pin_19), U1.43 (P1.0)
- new net 44: J8.20 (Pin_20), U1.44 (P1.1)
- new net 45: J8.21 (Pin_21), U1.45 (P1.2)
- new net 46: J8.22 (Pin_22), U1.46 (P1.3)
- new net 47: J8.23 (Pin_23), U1.47 (P1.4)
- new net 48: J8.24 (Pin_24), U1.48 (P1.5)
- new net 5: J7.5 (Pin_5), U1.5 (P4.5)
- new net 6: J7.6 (Pin_6), U1.6 (P4.4)
- new net 7: J7.7 (Pin_7), U1.7 (P3.1)
- new net 8: J7.8 (Pin_8), U1.8 (P3.2)
- new net 9: J7.9 (Pin_9), U1.9 (P3.3)
- new net BOOT: J7.16 (Pin_16), R7.2, SW2.2, U1.16 (P4.6)
- new net D0+: J2.3 (D+), J8.7 (Pin_7), SW3.5 (B), U1.31 (DP0)
- new net D0-: J2.2 (D-), J8.8 (Pin_8), SW3.2 (B), U1.32 (DM0)
- new net D1+: J3.3 (D+), J8.5 (Pin_5), U1.29 (DP1)
- new net D1-: J3.2 (D-), J8.6 (Pin_6), U1.30 (DM1)
- new net GND: C1.2, C2.2, C3.1, C4.2, C5.2, C6.2, C7.1, D1.1 (K), D2.1 (K), D3.1 (K), J1.A1 (GND), J1.A12 (GND), J1.B1 (GND), J1.B12 (GND), J1.S1 (SHIELD), J2.4 (GND), J2.5 (Shield), J3.4 (GND), J3.5 (Shield), J4.4 (Pin_4), J7.18 (Pin_18), R1.2, R2.2, R6.2, SW2.1, U1.18 (GND), U2.2 (GND)
- new net RST: J7.3 (Pin_3), R6.1, SW1.1, U1.3 (RST)
- new net VBUS: C1.1, C2.1, C3.2, C5.1, C7.2, D4.1 (K), J1.A4 (VBUS), J1.A9 (VBUS), J1.B4 (VBUS), J1.B9 (VBUS), J2.1 (VBUS), J3.1 (VBUS), J8.17 (Pin_17), U1.41 (VIN5), U2.1 (IN)
- new net aD0+: J1.A6 (D+), J1.B6 (D+), SW3.4 (A)
- new net aD0-: J1.A7 (D-), J1.B7 (D-), SW3.3 (C)
- no-connect marks 0 -> 4
