File: project/motor-driver/bldc-v1/bldc-v1.kicad_pcb (KiCad board)
At the start: 2 copper layers, 73.5 x 40 mm, 47 parts, among them J1 Power, J2 Input, J3 Output, Q1 NMOS, Q2 NMOS, Q3 NMOS, Q4 NMOS, Q5 NMOS, Q6 NMOS, U1 IR2302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

Commit message: 2025/12/13/11:43
Parts:
- added H1: MountingHole, MountingHole:MountingHole_3.2mm_M3, F.Cu at (184.0, 84.5)
- added H2: MountingHole, MountingHole:MountingHole_3.2mm_M3, F.Cu at (182.0, 112.5)
- added H3: MountingHole, MountingHole:MountingHole_3.2mm_M3, F.Cu at (134.0, 84.5)
- added H4: MountingHole, MountingHole:MountingHole_3.2mm_M3, F.Cu at (129.0, 120.0)
- moved J1 2.06 mm to (129.5, 106.0)
- moved J2 2.06 mm to (125.3, 83.0)
