File: project/motor-driver/bldc-v1/bldc-v1.kicad_sch (KiCad schematic)
At the start: 0 parts

Commit message: 2025/10/20/12:23
Parts:
- added C1, C4, C6: 1uF, Capacitor_SMD:C_0805_2012Metric, symbol Device:C
- added C10: 47uF, Capacitor_THT:CP_Radial_D6.3mm_P2.50mm, symbol Device:C_Polarized
- added C2, C3, C5: 0.1uF, Capacitor_SMD:C_0603_1608Metric, symbol Device:C
- added C9: 100uF, Capacitor_THT:CP_Radial_D8.0mm_P3.50mm, symbol Device:C_Polarized
- added D1, D2, D3: 1N4148W, Diode_SMD:D_SOD-123, symbol Diode:1N4148W
- added J1: Power, Connector_AMASS:AMASS_XT30PW-M_1x02_P2.50mm_Horizontal, symbol Connector:Conn_01x02_Socket
- added J2: Input, Connector_JST:JST_XH_S7B-XH-A_1x07_P2.50mm_Horizontal, symbol Connector:Conn_01x07_Pin
- added J3: Output, Connector_AMASS:AMASS_MR30PW-FB_1x03_P3.50mm_Horizontal, symbol Connector:Conn_01x03_Socket
- added Q1, Q2, Q3, Q4, Q5, Q6: NMOS, Package_TO_SOT_SMD:TO-252-2, symbol Transistor_FET_Other:Q_NMOS_Depletion_GDS
- added R1, R10, R3, R5, R6, R9: 10Ω, Resistor_SMD:R_0603_1608Metric, symbol Device:R
- added R11, R12, R13, R14, R15, R16, R17, R18, R2, R4, R7, R8: 10kΩ, Resistor_SMD:R_0603_1608Metric, symbol Device:R
- added R19, R20, R21, R22, R23, R24: 1kΩ, Resistor_SMD:R_0603_1608Metric, symbol Device:R
- added U1, U2, U3: IR2302, Package_SO:SOIC-8_3.9x4.9mm_P1.27mm, symbol Driver_FET:IR2302
Connections:
- new net: J2.6 (Pin_6), R14.1, R20.1
- new net: Q2.1 (G), R3.2, R4.2
- new net: R1.1, U1.7 (HO)
- new net: Q1.1 (G), R1.2, R2.2
- new net: R10.1, U3.5 (LO)
- new net: Q6.1 (G), R10.2, R12.2
- new net: C1.1, D1.1 (K), U1.8 (VB)
- new net: C4.1, D2.1 (K), U2.8 (VB)
- new net: R9.1, U3.7 (HO)
- new net: C6.1, D3.1 (K), U3.8 (VB)
- new net: J2.3 (Pin_3), R17.1, R23.1
- new net: J2.2 (Pin_2), R18.1, R24.1
- new net: J2.5 (Pin_5), R15.1, R21.1
- new net: J2.4 (Pin_4), R16.1, R22.1
- new net: Q5.1 (G), R11.2, R9.2
- new net: R5.1, U2.7 (HO)
- new net: Q3.1 (G), R5.2, R7.2
- new net: R3.1, U1.5 (LO)
- new net: J2.7 (Pin_7), R13.1, R19.1
- new net: R6.1, U2.5 (LO)
- new net: Q4.1 (G), R6.2, R8.2
- new net +12V: C10.1, C2.1, C3.1, C5.1, C9.1, D1.2 (A), D2.2 (A), D3.2 (A), J1.2 (Pin_2), Q1.2 (D), Q3.2 (D), Q5.2 (D), U1.1 (VCC), U2.1 (VCC), U3.1 (VCC)
- new net GND: C10.2, C2.2, C3.2, C5.2, C9.2, J1.1 (Pin_1), J2.1 (Pin_1), Q2.3 (S), Q4.3 (S), Q6.3 (S), R12.1, R13.2, R14.2, R15.2, R16.2, R17.2, R18.2, R4.1, R8.1, U1.4 (COM), U2.4 (COM), U3.4 (COM)
- new net IN_U: R20.2, U1.2 (IN)
- new net IN_V: R22.2, U2.2 (IN)
- new net IN_W: R24.2, U3.2 (IN)
- new net OUTPUT_U: C1.2, J3.1 (Pin_1), Q1.3 (S), Q2.2 (D), R2.1, U1.6 (VS)
- new net OUTPUT_V: C4.2, J3.2 (Pin_2), Q3.3 (S), Q4.2 (D), R7.1, U2.6 (VS)
- new net OUTPUT_W: C6.2, J3.3 (Pin_3), Q5.3 (S), Q6.2 (D), R11.1, U3.6 (VS)
- new net SD_U: R19.2, U1.3 (~{SD})
- new net SD_V: R21.2, U2.3 (~{SD})
- new net SD_W: R23.2, U3.3 (~{SD})

Commit message: 2025/12/13/11:43
Parts:
- added H1, H2, H3, H4: MountingHole, MountingHole:MountingHole_3.2mm_M3, symbol Mechanical:MountingHole

Commit message: 2026/04/22/08:58
Parts:
- removed C10: 47uF, Capacitor_THT:CP_Radial_D6.3mm_P2.50mm, symbol Device:C_Polarized
- removed C9: 100uF, Capacitor_THT:CP_Radial_D8.0mm_P3.50mm, symbol Device:C_Polarized
- removed D1, D2, D3: 1N4148W, Diode_SMD:D_SOD-123, symbol Diode:1N4148W
- removed H1, H2, H3, H4: MountingHole, MountingHole:MountingHole_3.2mm_M3, symbol Mechanical:MountingHole
- removed J2: Input, Connector_JST:JST_XH_S7B-XH-A_1x07_P2.50mm_Horizontal, symbol Connector:Conn_01x07_Pin
- removed J3: Output, Connector_AMASS:AMASS_MR30PW-FB_1x03_P3.50mm_Horizontal, symbol Connector:Conn_01x03_Socket
- removed R14: 10kΩ, Resistor_SMD:R_0603_1608Metric, symbol Device:R
- added C10: 1uF, symbol Device:C
- added C11: 0.01uF, symbol Device:C
- added C12, C13, C16, C18, C8, C9: 0.1uF, symbol Device:C
- added C14, C15: 20pF, symbol Device:C
- added C17: 0.22uF, symbol Device:C
- added C19, C20, C21, C22: C, symbol Device:C
- added C7: 4.7uF, symbol Device:C
- added D1, D2, D3, D4, D5: CUHS20S60, Diode_SMD:D_SOD-323, symbol Device:D_Schottky
- added FB1: FerriteBead, symbol Device:FerriteBead
- added J2: CAN, symbol Connector:Conn_01x02_Socket
- added J3: Encoder, symbol Connector:Conn_01x05_Socket
- added J4: Output, symbol Connector:Conn_01x03_Socket
- added J5: Debug, symbol Connector:Conn_01x05_Socket
- added J6: Limit_A, symbol Connector:Conn_01x02_Socket
- added J7: Limit_B, symbol Connector:Conn_01x02_Socket
- added L1, L2: L, symbol Device:L
- added R14: 5mΩ, symbol Device:R_Shunt
- added R25, R26: 1kΩ, symbol Device:R
- added R27, R28, R29, R30: R, symbol Device:R
- added SW1: Set_ID, symbol Switch:SW_DIP_x04
- added U4: STM32F303K8Tx, Package_QFP:LQFP-32_7x7mm_P0.8mm, symbol MCU_ST_STM32F3:STM32F303K8Tx
- added U5: MCP2562-E-SN, Package_SO:SOIC-8_3.9x4.9mm_P1.27mm, symbol Interface_CAN_LIN:MCP2562-E-SN
- added U6: NJM12888, Package_TO_SOT_SMD:SOT-23-5, symbol JRC_Regulator_Linear:NJM12888F33
- added U7: INA180B1, Package_TO_SOT_SMD:SOT-23-5, symbol Amplifier_Current:INA180B1
- added U8, U9: XC9704B75CPR-G, Package_TO_SOT_SMD:SOT-89-5, symbol TOREX_Regulator_switching:XC9704B75CPR-G
- added Y1: 16MHz, symbol Device:Crystal
- J1: footprint Connector_AMASS:AMASS_XT30PW-M_1x02_P2.50mm_Horizontal -> (none)
- Q1, Q2, Q3, Q4, Q5, Q6: value NMOS -> MTB7D0N6RJ3
- R13, R16, R17, R18: footprint Resistor_SMD:R_0603_1608Metric -> (none)
- R15: value 10kΩ -> 0Ω; footprint Resistor_SMD:R_0603_1608Metric -> (none)
- R19, R20, R21, R22, R23, R24: value 1kΩ -> 10kΩ; footprint Resistor_SMD:R_0603_1608Metric -> (none)
Connections:
- net GND: now also R13.1, R15.1, R19.2, R20.2, R21.2, R22.2, C12.2, C13.2, C14.1, C15.1, C16.2, C17.2, C18.2, C19.2, C20.2, C21.2, C22.2, C7.2, C8.2, C9.2, D4.2 (A), D5.2 (A), J3.1 (Pin_1), J5.1 (Pin_1), J6.1 (Pin_1), J7.1 (Pin_1), R28.1, R29.1, U4.16 (VSS), U4.32 (VSS), U5.2 (VSS), U5.8 (STBY), U6.2 (GND), U8.2 (GND), U9.2 (GND); no longer R13.2, R15.2
- net IN_U: no longer R20.2
- net IN_V: no longer R22.2
- net IN_W: no longer R24.2
- net OUTPUT_U: now also J4.3 (Pin_3)
- net OUTPUT_V: now also J4.2 (Pin_2)
- net OUTPUT_W: now also J4.1 (Pin_1)
- net SD_U: no longer R19.2
- net SD_V: no longer R21.2
- net SD_W: no longer R23.2
- net ENC_B: now reaches R20.1
- net ENC_B: now also J3.5 (Pin_5)
- net at C1.1, U1.8 (VB): now also D1.1 (K)
- net at C4.1, U2.8 (VB): now also D2.1 (K)
- net at C6.1, U3.8 (VB): now also D3.1 (K)
- net +3.3V: now reaches R23.1
- net +3.3V: now also R24.1, C13.1, C17.1, C7.1, C8.1, C9.1, FB1.1, J5.5 (Pin_5), SW1.1, SW1.2, SW1.3, SW1.4, U4.1 (VDD), U4.17 (VDD), U5.5 (Vio), U6.5 (Vout); no longer R17.1
- net ID2: now reaches R18.1
- net ID2: now also SW1.6; no longer R24.1
- net ENC_A: now reaches R21.1
- net ENC_A: now also J3.3 (Pin_3); no longer R15.1
- net ENC_Z: now reaches R22.1
- net ENC_Z: now also J3.2 (Pin_2); no longer R16.1
- net ID3: now reaches R19.1
- net ID3: now also SW1.5; no longer R13.1
- net +12V renamed +9V
- net +9V: now also C19.1, D1.2 (A), D2.2 (A), D3.2 (A), L1.2, R27.1; no longer J1.2 (Pin_2), Q1.2 (D), Q3.2 (D), Q5.2 (D)
- new net: R29.2, R30.2, U9.3 (FB)
- new net: R14.2, U7.1 (+)
- new net: R14.3, U7.3 (-)
- new net: D4.1 (K), L1.1, U8.1 (Lx)
- new net: R27.2, R28.2, U8.3 (FB)
- new net: D5.1 (K), L2.1, U9.1 (Lx)
- new net: J5.4 (Pin_4), R25.1
- new net: J5.3 (Pin_3), R26.1
- new net +3.3VA: C10.1, C11.1, C18.1, FB1.2, U4.5 (VDDA), U7.5 (V+)
- new net +5V: C12.1, C16.1, C22.1, J3.4 (Pin_4), L2.2, R30.1, U5.3 (VDD), U6.1 (Vin), U6.3 (Control)
- new net +BATT: C20.1, C21.1, J1.2 (Pin_2), R14.1, U8.4 (EN/SS), U8.5 (VIN), U9.4 (EN/SS), U9.5 (VIN)
- new net BOOT0: R13.2, U4.31 (BOOT0)
- new net CAN+: J2.2 (Pin_2), U5.7 (CANH)
- new net CAN-: J2.1 (Pin_1), U5.6 (CANL)
- new net CAN_RX: U4.21 (PA11), U5.4 (RXD)
- new net CAN_TX: U4.22 (PA12), U5.1 (TXD)
- new net CURRENT_OUTPUT: U7.4
- new net GNDA: C10.2, C11.2, R15.2, U7.2 (GND)
- new net ID0: R16.1, SW1.8
- new net ID1: R17.1, SW1.7
- new net LIMIT_A: J6.2 (Pin_2), R23.2
- new net LIMIT_B: J7.2 (Pin_2), R24.2
- new net MOTOR_PWR: Q1.2 (D), Q3.2 (D), Q5.2 (D), R14.4
- new net NRST: J5.2 (Pin_2), U4.4 (NRST)
- new net OSC_IN: C14.2, U4.2 (PF0), Y1.2
- new net OSC_OUT: C15.2, U4.3 (PF1), Y1.1
- new net SWCLK: R25.2, U4.24 (PA14)
- new net SWDIO: R26.2, U4.23 (PA13)
- no-connect marks 0 -> 20
Other:
- note added: "5mΩ * 30A = 0.15V 20倍なので 0.15V * 20 = 3V"
- moved on the sheet: C1, C2, C3, C4, C5, C6, Q1, Q2, Q3, Q4, Q5, Q6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

Commit message: 2026/04/23/17:05
Parts:
- removed D4, D5: CUHS20S60, Diode_SMD:D_SOD-323, symbol Device:D_Schottky
Other:
- moved on the sheet: C19, C21, C22, L1, L2, R27, R29, R30, U9

Commit message: 2026/05/01/16:47
Parts:
- removed C18: 0.1uF, symbol Device:C
- removed C21, C22: C, symbol Device:C
- removed D1, D2, D3: CUHS20S60, Diode_SMD:D_SOD-323, symbol Device:D_Schottky
- removed J5: Debug, symbol Connector:Conn_01x05_Socket
- removed J6: Limit_A, symbol Connector:Conn_01x02_Socket
- removed J7: Limit_B, symbol Connector:Conn_01x02_Socket
- removed Q1, Q2, Q3, Q4, Q5, Q6: MTB7D0N6RJ3, Package_TO_SOT_SMD:TO-252-2, symbol Transistor_FET_Other:Q_NMOS_Depletion_GDS
- removed R14: 5mΩ, symbol Device:R_Shunt
- removed R15: 0Ω, symbol Device:R
- removed R16, R17, R18, R19, R23, R24: 10kΩ, symbol Device:R
- removed R25, R26: 1kΩ, symbol Device:R
- removed R27, R29, R30: R, symbol Device:R
- removed SW1: Set_ID, symbol Switch:SW_DIP_x04
- removed U7: INA180B1, Package_TO_SOT_SMD:SOT-23-5, symbol Amplifier_Current:INA180B1
- removed U9: XC9704B75CPR-G, Package_TO_SOT_SMD:SOT-89-5, symbol TOREX_Regulator_switching:XC9704B75CPR-G
- added C2, C4, C6, C7: C, Capacitor_SMD:C_1210_3225Metric, symbol Device:C
- added D1, D2, D3: 1N4148W, Diode_SMD:D_SOD-123, symbol Diode:1N4148W
- added Q1, Q2, Q3, Q4, Q5, Q6: BSC030N08NS5, Package_TO_SOT_SMD:TDSON-8-1, symbol Transistor_FET:BSC030N08NS5
- added R4, R6, R7: R, Resistor_SMD:R_0603_1608Metric, symbol Device:R
- added U2: XC9704B75CPR-G, Package_TO_SOT_SMD:SOT-89-5, symbol TOREX_Regulator_switching:XC9704B75CPR-G
- C1: renamed from C20; footprint (none) -> Capacitor_SMD:C_1210_3225Metric
- C10: renamed from C17; footprint (none) -> Capacitor_SMD:C_0603_1608Metric
- C11: renamed from C7; footprint (none) -> Capacitor_SMD:C_0603_1608Metric
- C12: renamed from C13; footprint (none) -> Capacitor_SMD:C_0603_1608Metric
- C13: renamed from C8; footprint (none) -> Capacitor_SMD:C_0603_1608Metric
- C14: renamed from C12; footprint (none) -> Capacitor_SMD:C_0603_1608Metric
- C15: renamed from C9; footprint (none) -> Capacitor_SMD:C_0603_1608Metric
- C16: renamed from C10; footprint (none) -> Capacitor_SMD:C_0603_1608Metric
- C17: renamed from C11; footprint (none) -> Capacitor_SMD:C_0603_1608Metric
- C3: renamed from C19; footprint (none) -> Capacitor_SMD:C_1210_3225Metric
- C5: renamed from C16; footprint (none) -> Capacitor_SMD:C_0603_1608Metric
- C8: renamed from C14; footprint (none) -> Capacitor_SMD:C_0603_1608Metric
- C9: renamed from C15; footprint (none) -> Capacitor_SMD:C_0603_1608Metric
- FB1: value FerriteBead -> BLM18R; footprint (none) -> Inductor_SMD:L_0603_1608Metric
- J1: footprint (none) -> Connector_AMASS:AMASS_XT30PW-M_1x02_P2.50mm_Horizontal
- J2: footprint (none) -> Connector_JST:JST_XH_S2B-XH-A_1x02_P2.50mm_Horizontal
- J3: footprint (none) -> Connector_JST:JST_XH_S5B-XH-A_1x05_P2.50mm_Horizontal
- J4: footprint (none) -> Connector_AMASS:AMASS_MR30PW-FB_1x03_P3.50mm_Horizontal
- L1, L2: footprint (none) -> Inductor_SMD:L_1210_3225Metric
- R1: renamed from R20; footprint (none) -> Resistor_SMD:R_0603_1608Metric
- R2: renamed from R21; footprint (none) -> Resistor_SMD:R_0603_1608Metric
- R3: renamed from R22; footprint (none) -> Resistor_SMD:R_0603_1608Metric
- R5: renamed from R28; footprint (none) -> Resistor_SMD:R_0603_1608Metric
- R8: renamed from R13; footprint (none) -> Resistor_SMD:R_0603_1608Metric
- Y1: footprint (none) -> Crystal:Crystal_HC49-4H_Vertical
- renumbered C2 to C18, C3 to C19, C5 to C20, C1 to C21, C4 to C22, C6 to C23, R3 to R10, R5 to R11, R6 to R12, R9 to R13, R10 to R14, R2 to R15, R4 to R16, R7 to R17, R8 to R18, R11 to R19, R12 to R20, R1 to R9, U8 to U1, U6 to U3, U1 to U6, U2 to U7, U3 to U8
Connections:
- net GNDA is gone; now on net GND: C16.2, C17.2
- net +5V: now also C4.1, C7.1, R6.2
- net +9V: now also C6.1, D1.2 (A), D2.2 (A), D3.2 (A), R4.2
- net +BATT: now also C2.1, U2.4 (EN/SS), U2.5 (VIN)
- net GND: now also C2.2, C4.2, C6.2, C7.2, Q2.1 (S), Q2.2 (S), Q2.3 (S), Q4.1 (S), Q4.2 (S), Q4.3 (S), Q6.1 (S), Q6.2 (S), Q6.3 (S), R7.1, U2.2 (GND)
- net MOTOR_PWR: now also Q1.5 (D), Q3.5 (D), Q5.5 (D)
- net OUTPUT_U: now also Q1.1 (S), Q1.2 (S), Q1.3 (S), Q2.5 (D)
- net OUTPUT_V: now also Q3.1 (S), Q3.2 (S), Q3.3 (S), Q4.5 (D)
- net OUTPUT_W: now also Q5.1 (S), Q5.2 (S), Q5.3 (S), Q6.5 (D)
- net at R10.2, R16.2: now also Q2.4 (G)
- net at C22.1, U7.8 (VB): now also D2.1 (K)
- net at R15.2, R9.2: now also Q1.4 (G)
- net at R14.2, R20.2: now also Q6.4 (G)
- net at C23.1, U8.8 (VB): now also D3.1 (K)
- net at R5.2, U1.3 (FB): now also R4.1
- net at R13.2, R19.2: now also Q5.4 (G)
- net at R11.2, R17.2: now also Q3.4 (G)
- net at C21.1, U6.8 (VB): now also D1.1 (K)
- net at R12.2, R18.2: now also Q4.4 (G)
- net at L2.1: now also U2.1 (Lx)
- new net: R6.1, R7.2, U2.3 (FB)
Other:
- note removed: "5mΩ * 30A = 0.15V 20倍なので 0.15V * 20 = 3V"
- moved on the sheet: C1, C10, C11, C12, C13, C14, C15, C16, C17, C18, C19, C20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
