File: project/hobbies/f303k8-led-matrix-4layer/f303k8-led-matrix-4layer.kicad_sch (KiCad schematic)
At the start: 103 parts, among them J1 USB_C_Receptacle_USB2.0_16P, J2 Boot, U1 USBLC6-2SC6, U2 CH552E, U3 CH213K, U4 STM32F303K8Tx, U5 NJM12888

Commit message: 2026/01/30/13:22
Parts:
- renumbered D17 to D10, D4 to D11, D6 to D12, D8 to D13, D10 to D14, D12 to D15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
