File: project/motor-driver/dc-for-385-v1/dc-for-385-v1.kicad_pcb (KiCad board)
At the start: 2 copper layers, 32 x 36 mm, 44 parts, among them M1 RS385, Q1 TJ8S06M3L, U1 TB67H450FNG, U2 AP7375, U3 74AHC1G08, U4 74AHC1G08, U5 74AHC1G04

Commit message: 2026/01/30/13:22
Parts:
- added C19: 1000pF, Capacitor_SMD:C_0402_1005Metric, F.Cu at (149.1, 107.8)
- added R7: 1kΩ, Resistor_SMD:R_0603_1608Metric, F.Cu at (153.5, 113.1)
- added R8: 1kΩ, Resistor_SMD:R_0603_1608Metric, F.Cu at (152.0, 113.1)
- moved C11 3.29 mm to (160.8, 104.0)
- moved R5 2.02 mm to (163.5, 104.2), turned to -90 degrees
- moved U2 1.81 mm to (157.5, 103.3)
- moved D1 1.25 mm to (150.6, 106.2)
- moved D2 1.00 mm to (150.6, 109.5)
- moved R6 1.00 mm to (165.0, 103.2)
- moved D4 0.90 mm to (156.4, 112.5)
- moved Q1 0.71 mm to (142.2, 107.2)
- moved D3 0.25 mm to (135.8, 107.2)
Connections:
- D4 pad 1: PWM -> Net-(D4-A1)
- D4 pad 2: DIR -> Net-(D4-A2)
- R2 pad 1: DIR -> Net-(D4-A2)
- R3 pad 1: PWM -> Net-(D4-A1)
- TP3 pad 1: DIR -> Net-(D4-A2)
- TP4 pad 1: PWM -> Net-(D4-A1)
Routing:
- net DIR: track 23.3 -> 9.51 mm, vias 4 -> 0
- net Net-(D4-A2): track 0.00 -> 12.3 mm
- net PWM: track 27.0 -> 15.5 mm, vias 2 -> 3
- net Net-(D4-A1): track 0.00 -> 9.85 mm
- net +3.3V: track 28.8 -> 31.6 mm
- net Net-(D2-A): track 4.61 -> 7.11 mm
- net +BATT: track 35.9 -> 38.2 mm
- net Net-(D6-A): track 18.7 -> 16.4 mm
- net IN2: track 14.1 -> 12.2 mm
- net IN1: track 18.7 -> 20.4 mm
- net MOTOR_A: track 29.0 -> 30.0 mm
- net Net-(D5-K): track 13.2 -> 12.4 mm
- net MOTOR_B: track 55.3 -> 54.8 mm
- net GND: vias 137 -> 183
