File: project/motor-driver/dc-for-385-v1/dc-for-385-v1.kicad_sch (KiCad schematic)
At the start: 44 parts, among them M1 RS385, Q1 TJ8S06M3L, U1 TB67H450FNG, U2 AP7375, U3 74AHC1G08, U4 74AHC1G08, U5 74AHC1G04

Commit message: 2026/01/30/13:22
Parts:
- added C19: 1000pF, Capacitor_SMD:C_0402_1005Metric, symbol Device:C
- added R7, R8: 1kΩ, Resistor_SMD:R_0603_1608Metric, symbol Device:R
Connections:
- net +BATT: now also C19.1
- net DIR: now also R7.2; no longer D4.2 (A2), R2.1, TP3.1
- net PWM: now also R8.2; no longer D4.1 (A1), R3.1, TP4.1
- net at D2.2 (A), Q1.1 (G), R1.1: now also C19.2
- new net: D4.2 (A2), R2.1, R7.1, TP3.1
- new net: D4.1 (A1), R3.1, R8.1, TP4.1
