File: project/robocon/can-tranceiver-module/can-tranceiver-module.kicad_sch (KiCad schematic)
At the start: 12 parts, among them J1 Conn_01x07_Pin, SW1 SlideSwitch, U1 MCP2562-E-P, U2 AZ1117-3.3

Commit message: 2026/03/23/22:21
Connections:
- net +3.3V: now also D1.2 (A); no longer R1.1
- net GND: now also R1.1; no longer D1.1 (K)
- net at R1.2: now also D1.1 (K); no longer D1.2 (A)
Other:
- moved on the sheet: D1, R1
Changed lines of the file:
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@@
 	(symbol
 		(lib_id "Device:R")
-		(at 153.67 64.77 0)
+		(at 153.67 73.66 180)
 		(unit 1)
 		(exclude_from_sim no)
@@
 		(fields_autoplaced yes)
 		(property "Reference" "R1"
-			(at 156.21 63.4999 0)
-			(effects
-				(font
-					(size 1.27 1.27)
-				)
-				(justify left)
+			(at 156.21 72.3899 0)
+			(effects
+				(font
+					(size 1.27 1.27)
+				)
+				(justify right)
 			)
 		)
 		(property "Value" "1kΩ"
-			(at 156.21 66.0399 0)
-			(effects
-				(font
-					(size 1.27 1.27)
-				)
-				(justify left)
+			(at 156.21 74.9299 0)
+			(effects
+				(font
+					(size 1.27 1.27)
+				)
+				(justify right)
 			)
 		)
 		(property "Footprint" "Resistor_THT:R_Axial_DIN0207_L6.3mm_D2.5mm_P10.16mm_Horizontal"
-			(at 151.892 64.77 90)
+			(at 155.448 73.66 90)
 			(effects
 				(font
@@
 		)
 		(property "Datasheet" "~"
-			(at 153.67 64.77 0)
+			(at 153.67 73.66 0)
 			(effects
 				(font
@@
 		)
 		(property "Description" "Resistor"
-			(at 153.67 64.77 0)
+			(at 153.67 73.66 0)
 			(effects
 				(font
@@
 	(symbol
 		(lib_id "Device:LED")
-		(at 153.67 73.66 90)
+		(at 153.67 64.77 90)
 		(unit 1)
 		(exclude_from_sim no)
@@
 		(fields_autoplaced yes)
 		(property "Reference" "D1"
-			(at 157.48 73.9774 90)
+			(at 157.48 65.0874 90)
 			(effects
 				(font
@@
 		)
 		(property "Value" "GREEN"
-			(at 157.48 76.5174 90)
+			(at 157.48 67.6274 90)
 			(effects
 				(font
@@
 		)
 		(property "Footprint" "LED_THT:LED_D5.0mm"
-			(at 153.67 73.66 0)
+			(at 153.67 64.77 0)
 			(effects
 				(font
@@
 		)
 		(property "Datasheet" "~"
-			(at 153.67 73.66 0)
+			(at 153.67 64.77 0)
 			(effects
 				(font
@@
 		)
 		(property "Description" "Light emitting diode"
-			(at 153.67 73.66 0)
+			(at 153.67 64.77 0)
 			(effects
 				(font
@@
 		)
 		(property "Sim.Pins" "1=K 2=A"
-			(at 153.67 73.66 0)
-			(effects
-				(font
+			(at 153.67 64.77 0)
+			(effects
+				(font

Commit message: 2026/03/25/15:21
Parts:
- removed U2: AZ1117-3.3, Package_TO_SOT_SMD:SOT-223-3_TabPin2, symbol Regulator_Linear:AZ1117-3.3
- added R4: 6.1kΩ, Resistor_SMD:R_0603_1608Metric, symbol Device:R
- added R5: 10kΩ, Resistor_SMD:R_0603_1608Metric, symbol Device:R
- added U2: AZ1117H-ADJ, Package_TO_SOT_SMD:SOT-223-3_TabPin2, symbol Regulator_Linear:AZ1117H-ADJ
Connections:
- net +3.3V: now also R4.1, U2.2 (VO)
- net +5V: now also U2.3 (VI)
- net GND: now also R5.2
- new net: R4.2, R5.1, U2.1 (ADJ)
Other:
- moved on the sheet: C1, C2
