File: project/robocon/power-control-v1/power-control-v1.kicad_sch (KiCad schematic)
At the start: 0 parts

Commit message: 2026/04/22/08:58
Parts:
- added F1, F2: max30A, symbol Device:Fuse
- added J1: PWR_IN_24v, Connector_AMASS:AMASS_XT60PW-M_1x02_P7.20mm_Horizontal, symbol Connector:Conn_01x02_Socket
- added J2: PWR_IN_12v, Connector_AMASS:AMASS_XT30PW-M_1x02_P2.50mm_Horizontal, symbol Connector:Conn_01x02_Socket
- added J3, J4: EMS1, symbol Connector:Conn_01x02_Socket
- added J5: PWR_OUT_24v, Connector_AMASS:AMASS_XT60PW-M_1x02_P7.20mm_Horizontal, symbol Connector:Conn_01x02_Socket
- added J6: PWR_OUT_12v, Connector_AMASS:AMASS_XT60PW-M_1x02_P7.20mm_Horizontal, symbol Connector:Conn_01x02_Socket
- added SW1: MAIN_24v, symbol Switch:SW_SPST
- added SW2: MAIN_12v, symbol Switch:SW_SPST
- added TH1, TH2: Thermistor_NTC, symbol Device:Thermistor_NTC
Connections:
- new net: F2.1, TH2.2
- new net: F2.2, J4.1 (Pin_1)
- new net: J5.1 (Pin_1), SW1.2 (B)
- new net: J6.1 (Pin_1), SW2.2 (B)
- new net: J2.2 (Pin_2), TH2.1
- new net: F1.2, J3.1 (Pin_1)
- new net: J1.2 (Pin_2), TH1.1
- new net: F1.1, TH1.2
- new net +12V: J4.2 (Pin_2), SW2.1 (A)
- new net +24V: J3.2 (Pin_2), SW1.1 (A)
- new net GND: J1.1 (Pin_1), J2.1 (Pin_1), J5.2 (Pin_2), J6.2 (Pin_2)
