File: project/robocon/usb-can-bridge/usb-can-bridge.kicad_pcb (KiCad board)
At the start: 4 copper layers, 55 x 20 mm, 36 parts, among them J1 USB_A, J2 Debug, J3 CAN, J4 Reset, SW1 Boot, SW2 CAN_R_SW, U1 USBLC6-2SC6, U2 NJM12888, U3 CH340N, U4 STM32F303K8Tx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

Commit message: 2026/04/22/08:58
Routing:
- net GND: track 36.6 -> 37.6 mm, vias 105 -> 100
