File: project/motor-driver/dc-for-385-v2/dc-for-385-v2.kicad_pcb (KiCad board)
At the start: 2 copper layers, 51 x 25 mm, 44 parts, among them J1 Power, J2 Output, J3 Input, Q1 TPH11006NL, Q2 TPH11006NL, Q3 TPH11006NL, Q4 TPH11006NL, U1 IR2302, U2 IR2302, U3 L7808

Commit message: 2026/06/29/10:17
Routing:
- net IN_A: track 32.6 -> 34.7 mm
- net Net-(U1-LO): track 38.5 -> 37.1 mm
- net MOTOR_B: track 11.9 -> 11.0 mm, vias 27 -> 52
- net MOTOR_A: vias 27 -> 52
- net GND: vias 135 -> 171
- net +BATT: vias 111 -> 196
Other:
- board text added: "v1.0.1 @netetra07"
- board text removed: "v1.0.0 @netetra07"
