File: project/research/anything/anything.kicad_sch (KiCad schematic)
At the start: 0 parts

Commit message: 2026/07/14/12:02
Parts:
- added C1, C2, C3, C4, C5, C6: C, symbol Device:C
- added D1, D2, D3, D4, D5, D6: D, symbol Device:D
Connections:
- new net: C1.2, C3.1, D1.2 (A), D2.1 (K)
- new net: C2.2, C4.1, D2.2 (A), D3.1 (K)
- new net: C4.2, C6.1, D4.2 (A), D5.1 (K)
- new net: C2.1, D1.1 (K)
- new net: C3.2, C5.1, D3.2 (A), D4.1 (K)
- new net: C5.2, D5.2 (A), D6.1 (K)
- new net: C6.2, D6.2 (A)
