File: project/robocon/can-power-hub/can-power-hub.kicad_pcb (KiCad board)
At the start: 2 copper layers, 85 x 25 mm, 12 parts, among them J1 Connector, J2 Connector, J3 Connector, J4 Connector, J5 Connector, J6 Connector

Commit message: 2026/07/16/16:32
Other:
- board text added: "CAN_L CAN_H GND 5V"
Changed lines of the file:
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@@
 		(layer "Edge.Cuts")
+	)
+	(gr_text "CAN_L\nCAN_H\nGND\n5V"
+		(at 41.5 107 0)
+		(layer "B.SilkS")
+		(effects
+			(font
+				(size 1.5 1.5)
+				(thickness 0.25)
+				(bold yes)
+			)
+			(justify left mirror)
+		)
+	)
+	(gr_text "CAN_L\nCAN_H\nGND\n5V"
+		(at 111.5 107 180)
+		(layer "B.SilkS")
+		(effects
+			(font
+				(size 1.5 1.5)
+				(thickness 0.25)
+				(bold yes)
+			)
+			(justify left mirror)
+		)
+	)
+	(gr_text "CAN_L\nCAN_H\nGND\n5V"
+		(at 54 101.5 270)
+		(layer "B.SilkS")
+		(effects
+			(font
+				(size 1.5 1.5)
+				(thickness 0.25)
+				(bold yes)
+			)
+			(justify left mirror)
+		)
+	)
+	(gr_text "CAN_L\nCAN_H\nGND\n5V"
+		(at 69 101.5 270)
+		(layer "B.SilkS")
+		(effects
+			(font
+				(size 1.5 1.5)
+				(thickness 0.25)
+				(bold yes)
+			)
+			(justify left mirror)
+		)
+	)
+	(gr_text "CAN_L\nCAN_H\nGND\n5V"
+		(at 84 101.5 270)
+		(layer "B.SilkS")
+		(effects
+			(font
+				(size 1.5 1.5)
+				(thickness 0.25)
+				(bold yes)
+			)
+			(justify left mirror)
+		)
+	)
+	(gr_text "CAN_L\nCAN_H\nGND\n5V"
+		(at 99 101.5 270)
+		(layer "B.SilkS")
+		(effects
+			(font
+				(size 1.5 1.5)
+				(thickness 0.25)
+				(bold yes)
+			)
+			(justify left mirror)
+		)
 	)
 	(dimension
