File: project/robocon/esp32s3-main-v1/esp32s3-main-v1.kicad_pcb (KiCad board)
At the start: 4 copper layers, 34 x 56 mm, 19 parts, among them J1 PowerSupply & Programming, J2 CAN, J3 Controller, J4 GPIO, U1 XIAO-ESP32-S3-SMD, U2 MCP2562-E-SN, U3 USBLC6-2SC6, U4 USBLC6-2SC6, U5 CH340N

Commit message: 2026/07/16/16:32
Parts:
- added D1: LED, LED_SMD:LED_0603_1608Metric, F.Cu at (103.0, 57.0)
- added R4: 22Ω, Resistor_SMD:R_0603_1608Metric, F.Cu at (102.8, 87.2)
- added R5: 22Ω, Resistor_SMD:R_0603_1608Metric, F.Cu at (104.2, 87.2)
- added R6: 1kΩ, Resistor_SMD:R_0603_1608Metric, F.Cu at (99.0, 57.0)
Connections:
- U1 pad 21: ESP_D- -> 'ESP_D-
- U1 pad 22: ESP_D+ -> 'ESP_D+
Routing:
- net ESP_D+: track 24.4 -> 3.31 mm, vias 2 -> 0
- net ESP_D-: track 23.6 -> 3.31 mm, vias 2 -> 0
- net 'ESP_D+: track 0.00 -> 19.3 mm, vias 0 -> 2
- net 'ESP_D-: track 0.00 -> 18.5 mm, vias 0 -> 2
- net Net-(D1-A): track 0.00 -> 2.39 mm
- net GND: vias 27 -> 31
- net +5V: vias 7 -> 8
Other:
- board text added: "5V GND CAN_H CAN_L"
- board text added: "GND D10 D9 D8 D2 D3 D4 D5 5V"
- board text removed: "CAN"
- board text removed: "GPIO"
- board text removed: "Power"
- board text removed: "USB"
