File: project/hobbies/ruler/ruler.kicad_pcb (KiCad board)
At the start: 2 copper layers, 165 x 25 mm, 5 parts

Commit message: 2026/09/07/13:51
Parts:
- added ?: , , F.Cu at (84.2, 113.0)
- added ?: , , F.Cu at (85.0, 110.0)
- added ?: , , F.Cu at (85.0, 113.0)
- added ?: , , F.Cu at (81.5, 110.0)
- added ?: , , F.Cu at (85.1, 107.0)
- added ?: , , F.Cu at (82.5, 107.0)
- added ?: , , F.Cu at (85.4, 113.0)
- added ?: , , F.Cu at (89.0, 107.0)
- added ?: , , F.Cu at (82.6, 113.0)
- added ?: , , F.Cu at (83.2, 107.0)
- added ?: , , F.Cu at (86.0, 110.0)
- added ?: , , F.Cu at (81.8, 104.0)
- added ?: , , F.Cu at (84.6, 113.0)
- added ?: , , F.Cu at (81.8, 113.0)
- added ?: , , F.Cu at (83.8, 113.0)
- added ?: , , F.Cu at (88.2, 113.0)
- added ?: , , F.Cu at (85.2, 101.0)
- added ?: , , F.Cu at (87.7, 107.0)
- added ?: , , F.Cu at (87.8, 113.0)
- added ?: , , F.Cu at (83.5, 110.0)
- added ?: , , F.Cu at (85.0, 104.0)
- added ?: , , F.Cu at (86.5, 110.0)
- added ?: , , F.Cu at (85.8, 107.0)
- added ?: , , F.Cu at (88.5, 110.0)
- added ?: , , F.Cu at (88.3, 107.0)
- added ?: , , F.Cu at (81.2, 107.0)
- added ?: , , F.Cu at (86.6, 113.0)
- added ?: , , F.Cu at (87.0, 110.0)
- added ?: , , F.Cu at (82.0, 110.0)
- added ?: , , F.Cu at (87.5, 110.0)
- added ?: , , F.Cu at (85.8, 113.0)
- added ?: , , F.Cu at (84.5, 107.0)
- added ?: , , F.Cu at (85.8, 104.0)
- added ?: , , F.Cu at (81.4, 101.0)
- added ?: , , F.Cu at (88.0, 110.0)
- added ?: , , F.Cu at (86.2, 113.0)
- added ?: , , F.Cu at (83.8, 107.0)
- added ?: , , F.Cu at (83.0, 110.0)
- added ?: , , F.Cu at (82.2, 113.0)
- added ?: , , F.Cu at (85.5, 110.0)
- added ?: , , F.Cu at (87.0, 107.0)
- added ?: , , F.Cu at (81.4, 113.0)
- added ?: , , F.Cu at (83.4, 104.0)
- added ?: , , F.Cu at (84.5, 110.0)
- added ?: , , F.Cu at (87.0, 113.0)
- added ?: , , F.Cu at (89.0, 110.0)
- added ?: , , F.Cu at (82.7, 101.0)
- added ?: , , F.Cu at (89.0, 104.0)
- added ?: , , F.Cu at (84.0, 110.0)
- added ?: , , F.Cu at (88.6, 113.0)
- added ?: , , F.Cu at (89.0, 101.0)
- added ?: , , F.Cu at (84.2, 104.0)
- added ?: , , F.Cu at (88.2, 104.0)
- added ?: , , F.Cu at (82.6, 104.0)
- added ?: , , F.Cu at (83.4, 113.0)
- added ?: , , F.Cu at (83.0, 113.0)
- added ?: , , F.Cu at (86.6, 104.0)
- added ?: , , F.Cu at (87.4, 113.0)
- added ?: , , F.Cu at (82.5, 110.0)
- added ?: , , F.Cu at (87.4, 104.0)
- added ?: , , F.Cu at (89.0, 113.0)
- added ?: , , F.Cu at (87.7, 101.0)
- added ?: , , F.Cu at (86.5, 101.0)
- added ?: , , F.Cu at (86.4, 107.0)
- added ?: , , F.Cu at (81.8, 107.0)
- added ?: , , F.Cu at (83.9, 101.0)
- added REF**: C_1206_3216Metric, Capacitor_SMD:C_1206_3216Metric, F.Cu at (172.5, 106.5)
- added REF**: C_01005_0402Metric, Capacitor_SMD:C_01005_0402Metric, F.Cu at (148.5, 106.5)
- added REF**: C_1808_4520Metric, Capacitor_SMD:C_1808_4520Metric, F.Cu at (180.5, 106.5)
- added REF**: C_0504_1310Metric, Capacitor_SMD:C_0504_1310Metric, F.Cu at (160.5, 106.5)
- added REF**: C_0603_1608Metric, Capacitor_SMD:C_0603_1608Metric, F.Cu at (164.5, 106.5)
- added REF**: C_0402_1005Metric, Capacitor_SMD:C_0402_1005Metric, F.Cu at (156.5, 106.5)
- added REF**: C_0805_2012Metric, Capacitor_SMD:C_0805_2012Metric, F.Cu at (168.5, 106.5)
- added REF**: C_1210_3225Metric, Capacitor_SMD:C_1210_3225Metric, F.Cu at (176.5, 106.5)
- added REF**: C_0201_0603Metric, Capacitor_SMD:C_0201_0603Metric, F.Cu at (152.5, 106.5)
- added REF**9: C_1812_4532Metric, Capacitor_SMD:C_1812_4532Metric, F.Cu at (184.5, 106.5)
- moved 3.50 10.5 mm to (211.0, 108.0)
- moved 3.80 10.0 mm to (200.5, 107.9)
- moved 2.00 7.25 mm to (191.5, 102.5)
- moved 2.50 3.34 mm to (191.5, 110.7)
- renumbered 2.0mm to 2.00, 2.5mm to 2.50, 3.5mm to 3.50, 3.8mm to 3.80, 5.0mm to 5.00
Routing:
- net (no net): vias 0 -> 16
Other:
- board text added: "0.40"
- board text added: "0.50"
- board text added: "0.65"
- board text added: "0.80"
- board text added: "0201"
- board text added: "0402"
- board text added: "0504"
- board text added: "0603"
- board text added: "0805"
- board text added: "1.00"
- board text added: "1.27"
- board text added: "1005"
- board text added: "1206"
- board text added: "1210"
- board text added: "1310"
- board text added: "1608"
- board text added: "1808"
- board text added: "1812"
- board text added: "2.00"
- board text added: "2.54"
- board text added: "2012"
- board text added: "3216"
- board text added: "3225"
- board text added: "4520"
- board text added: "4532"
- board text added: "[inch/metric]"
