File: project/robocon/esp32s3-test-board/esp32s3-test-board.kicad_pcb (KiCad board)
At the start: 2 copper layers, 100 x 70 mm, 30 parts, among them J1 AMT22, J10 LimitSW, J11 LimitSW, J12 LimitSW, J13 GPIO, J14 GPIO, J15 C620, J16 C620, J17 C620, J18 Power&CAN, J19 mcp25625_breakout, J2 AMT22, J3 AMT22, J4 AMT102, J5 AMT102, J6 AMT102, J7 MD, J8 MD, J9 MD, U1 ESP32-S3-DevKitC, U2 MCP2562-E-P

Commit message: 2026/09/10/20:06
Parts:
- R1, R2, R3, R5: value R -> 1kΩ
