File: project/robocon/stm32f303-module/stm32f303-module.kicad_pcb (KiCad board)
At the start: 2 copper layers, 31.7 x 21.6 mm, 19 parts, among them J1 GPIO, J2 GPIO, U2 NJM12888, U4 STM32F303K8Tx, U5 MCP2562-E-SN, Y1 16MHz

Commit message: 2026/09/21/14:12
Parts:
- moved D1 0.25 mm to (157.8, 108.8)
- moved R1 0.25 mm to (154.8, 108.8)
Connections:
- J1 pad 1: unconnected-(J1-Pin_1-Pad1) -> PA0
- J1 pad 2: unconnected-(J1-Pin_2-Pad2) -> PA1
- J1 pad 3: unconnected-(J1-Pin_3-Pad3) -> PA4
Routing:
- net PA0: track 0.00 -> 14.1 mm
- net PA1: track 0.00 -> 11.2 mm
- net PA4: track 0.00 -> 10.6 mm
- net GND: vias 39 -> 48
- net +5V: vias 4 -> 2
