File: project/robocon/stm32f303-module/stm32f303-module.kicad_sch (KiCad schematic)
At the start: 3 parts, among them U1 STM32F303K8Tx, U2 MCP2562-E-SN, U3 NJM12888

Commit message: 2026/09/21/10:32
Parts:
- removed U1: STM32F303K8Tx, Package_QFP:LQFP-32_7x7mm_P0.8mm, symbol MCU_ST_STM32F3:STM32F303K8Tx
- removed U2: MCP2562-E-SN, Package_SO:SOIC-8_3.9x4.9mm_P1.27mm, symbol Interface_CAN_LIN:MCP2562-E-SN
- removed U3: NJM12888, Package_TO_SOT_SMD:SOT-23-5, symbol JRC_Regulator_Linear:NJM12888F33
- added C1, C10, C4, C5, C6, C9: 0.1uF, Capacitor_SMD:C_0603_1608Metric, symbol Device:C
- added C2: 0.22uF, Capacitor_SMD:C_0603_1608Metric, symbol Device:C
- added C3: 4.7uF, Capacitor_SMD:C_0603_1608Metric, symbol Device:C
- added C7, C8: 20pF, Capacitor_SMD:C_0603_1608Metric, symbol Device:C
- added D1: Blue, LED_SMD:LED_0603_1608Metric, symbol Device:LED
- added J1, J2: GPIO, Connector_PinHeader_2.54mm:PinHeader_1x12_P2.54mm_Vertical, symbol Connector:Conn_01x12_Pin
- added R1: 1kΩ, Resistor_SMD:R_0603_1608Metric, symbol Device:R
- added R4: 10kΩ, Resistor_SMD:R_0603_1608Metric, symbol Device:R
- added U2: NJM12888, Package_TO_SOT_SMD:SOT-23-5, symbol JRC_Regulator_Linear:NJM12888F33
- added U4: STM32F303K8Tx, Package_QFP:LQFP-32_7x7mm_P0.8mm, symbol MCU_ST_STM32F3:STM32F303K8Tx
- added U5: MCP2562-E-SN, Package_SO:SOIC-8_3.9x4.9mm_P1.27mm, symbol Interface_CAN_LIN:MCP2562-E-SN
- added Y1: 16MHz, Crystal:Crystal_HC49-4H_Vertical, symbol Device:Crystal
Connections:
- net +3.3V: now also C10.1, C2.1, C3.1, C4.1, C5.1, C6.1, R1.1, U2.5 (Vout), U4.1 (VDD), U4.17 (VDD), U4.5 (VDDA), U5.5 (Vio)
- net +5V: now also C1.1, C9.2, J1.12 (Pin_12), U2.1 (Vin), U2.3 (Control), U5.3 (VDD)
- net GND: now also C1.2, C10.2, C2.2, C3.2, C4.2, C5.2, C6.2, C7.1, C8.1, C9.1, D1.1 (K), J2.10 (Pin_10), R4.1, U2.2 (GND), U4.16 (VSS), U4.32 (VSS), U5.2 (VSS), U5.8 (STBY)
- new net: D1.2 (A), R1.2
- new net BOOT0: R4.2, U4.31 (BOOT0)
- new net CAN+: J2.11 (Pin_11), U5.7 (CANH)
- new net CAN-: J2.12 (Pin_12), U5.6 (CANL)
- new net CAN_RX: U4.21 (PA11), U5.4 (RXD)
- new net CAN_TX: U4.22 (PA12), U5.1 (TXD)
- new net NRST: J2.7 (Pin_7), U4.4 (NRST)
- new net OSC_IN: C7.2, U4.2 (PF0), Y1.2
- new net OSC_OUT: C8.2, U4.3 (PF1), Y1.1
- new net PA0: U4.6 (PA0)
- new net PA1: U4.7 (PA1)
- new net PA10: J1.11 (Pin_11), U4.20 (PA10)
- new net PA15: J2.6 (Pin_6), U4.25 (PA15)
- new net PA2: U4.8 (PA2)
- new net PA3: U4.9 (PA3)
- new net PA4: U4.10 (PA4)
- new net PA5: J1.4 (Pin_4), U4.11 (PA5)
- new net PA6: J1.5 (Pin_5), U4.12 (PA6)
- new net PA7: J1.6 (Pin_6), U4.13 (PA7)
- new net PA8: J1.9 (Pin_9), U4.18 (PA8)
- new net PA9: J1.10 (Pin_10), U4.19 (PA9)
- new net PB0: J1.7 (Pin_7), U4.14 (PB0)
- new net PB1: J1.8 (Pin_8), U4.15 (PB1)
- new net PB3: J2.5 (Pin_5), U4.26 (PB3)
- new net PB4: J2.4 (Pin_4), U4.27 (PB4)
- new net PB5: J2.3 (Pin_3), U4.28 (PB5)
- new net PB6: J2.2 (Pin_2), U4.29 (PB6)
- new net PB7: J2.1 (Pin_1), U4.30 (PB7)
- new net SWCLK: J2.8 (Pin_8), U4.24 (PA14)
- new net SWDIO: J2.9 (Pin_9), U4.23 (PA13)

Commit message: 2026/09/21/14:12
Connections:
- net PA0: now also J1.1 (Pin_1)
- net PA1: now also J1.2 (Pin_2)
- net PA4: now also J1.3 (Pin_3)
Changed lines of the file:
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@@
 	)
 	(junction
+		(at 228.6 71.12)
+		(diameter 0)
+		(color 0 0 0 0)
+	)
+	(junction
+		(at 251.46 66.04)
+		(diameter 0)
+		(color 0 0 0 0)
+	)
+	(junction
 		(at 153.67 60.96)
 		(diameter 0)
@@
 	(wire
 		(pts
-			(xy 229.87 71.12) (xy 218.44 71.12)
+			(xy 153.67 63.5) (xy 149.86 63.5)
 		)
 		(stroke
@@
 	(wire
 		(pts
-			(xy 153.67 63.5) (xy 149.86 63.5)
+			(xy 95.25 92.71) (xy 97.79 92.71)
 		)
 		(stroke
@@
 	(wire
 		(pts
-			(xy 95.25 92.71) (xy 97.79 92.71)
+			(xy 124.46 46.99) (xy 124.46 48.26)
 		)
 		(stroke
@@
 	(wire
 		(pts
-			(xy 124.46 46.99) (xy 124.46 48.26)
+			(xy 78.74 119.38) (xy 85.09 119.38)
 		)
 		(stroke
@@
 	(wire
 		(pts
-			(xy 78.74 119.38) (xy 85.09 119.38)
+			(xy 86.36 80.01) (xy 86.36 86.36)
 		)
 		(stroke
@@
 	(wire
 		(pts
-			(xy 86.36 80.01) (xy 86.36 86.36)
+			(xy 228.6 71.12) (xy 218.44 71.12)
 		)
 		(stroke
@@
 	(wire
 		(pts
-			(xy 229.87 69.85) (xy 229.87 71.12)
+			(xy 228.6 69.85) (xy 228.6 71.12)
 		)
 		(stroke
@@
 		)
 	)
-	(global_label "PA3"
-		(shape bidirectional)
-		(at 219.71 45.72 0)
-		(fields_autoplaced yes)
-		(effects
-			(font
-				(size 1.27 1.27)
-			)
-			(justify left)
-		)
-		(property "Intersheetrefs" "${INTERSHEET_REFS}"
-			(at 227.3746 45.72 0)
-			(hide yes)
-			(show_name no)
-			(do_not_autoplace no)
-			(effects
-				(font
-					(size 1.27 1.27)
-				)
-				(justify left)
-			)
-		)
-	)
 	(global_label "PA9"
 		(shape bidirectional)
@@
 	(global_label "PA4"
 		(shape bidirectional)
-		(at 219.71 48.26 0)
+		(at 218.44 48.26 0)
 		(fields_autoplaced yes)
 		(effects
@@
 		)
 		(property "Intersheetrefs" "${INTERSHEET_REFS}"
-			(at 227.3746 48.26 0)
+			(at 226.1046 48.26 0)
 			(hide yes)
 			(show_name no)
@@
 	(global_label "PA0"
 		(shape bidirectional)
-		(at 219.71 38.1 0)
+		(at 218.44 43.18 0)
 		(fields_autoplaced yes)
 		(effects
@@
 		)
 		(property "Intersheetrefs" "${INTERSHEET_REFS}"
-			(at 227.3746 38.1 0)
+			(at 226.1046 43.18 0)
 			(hide yes)
 			(show_name no)
@@
 		)
 	)
-	(global_label "PA2"
-		(shape bidirectional)
-		(at 219.71 43.18 0)
-		(fields_autoplaced yes)
-		(effects
-			(font
-				(size 1.27 1.27)
-			)
-			(justify left)
-		)
-		(property "Intersheetrefs" "${INTERSHEET_REFS}"
-			(at 227.3746 43.18 0)
-			(hide yes)
-			(show_name no)
-			(do_not_autoplace no)
-			(effects
-				(font
-					(size 1.27 1.27)
-				)
-				(justify left)
-			)
-		)
-	)
 	(global_label "SWDIO"
 		(shape bidirectional)
@@
 	(global_label "PA1"
 		(shape bidirectional)
-		(at 219.71 40.64 0)
+		(at 218.44 45.72 0)
 		(fields_autoplaced yes)
 		(effects
@@
 		)
 		(property "Intersheetrefs" "${INTERSHEET_REFS}"
-			(at 227.3746 40.64 0)
+			(at 226.1046 45.72 0)
 			(hide yes)
 			(show_name no)
@@
 	(symbol
 		(lib_id "power:+5V")
-		(at 229.87 69.85 0)
+		(at 228.6 69.85 0)
 		(unit 1)
 		(body_style 1)
@@
 		(fields_autoplaced yes)
 		(property "Reference" "#PWR07"
-			(at 229.87 73.66 0)
+			(at 228.6 73.66 0)
 			(hide yes)
 			(show_name no)
@@
 		)
 		(property "Value" "+5V"
-			(at 229.87 64.77 0)
+			(at 228.6 64.77 0)
 			(show_name no)
 			(do_not_autoplace no)
@@
 		)
 		(property "Footprint" ""
-			(at 229.87 69.85 0)
+			(at 228.6 69.85 0)
 			(hide yes)
 			(show_name no)
@@
 		)
 		(property "Datasheet" ""
-			(at 229.87 69.85 0)
+			(at 228.6 69.85 0)
 			(hide yes)
 			(show_name no)
@@
 		)
 		(property "Description" "Power symbol creates a global label with name \"+5V\""
-			(at 229.87 69.85 0)
+			(at 228.6 69.85 0)
 			(hide yes)
 			(show_name no)
@@
 	)
 	(symbol
+		(lib_id "power:PWR_FLAG")
+		(at 228.6 71.12 180)
+		(unit 1)
+		(body_style 1)
+		(exclude_from_sim no)
+		(in_bom yes)
+		(on_board yes)
+		(in_pos_files yes)
+		(dnp no)
+		(fields_autoplaced yes)
+		(property "Reference" "#FLG01"
+			(at 228.6 73.025 0)
+			(hide yes)
+			(show_name no)
+			(do_not_autoplace no)
+			(effects
+				(font
+					(size 1.27 1.27)
+				)
+			)
+		)
+		(property "Value" "PWR_FLAG"
+			(at 228.6 76.2 0)
+			(show_name no)
+			(do_not_autoplace no)
+			(effects
+				(font
+					(size 1.27 1.27)
+				)
+			)
+		)
+		(property "Footprint" ""
+			(at 228.6 71.12 0)
+			(hide yes)
+			(show_name no)
+			(do_not_autoplace no)
+			(effects
+				(font
+					(size 1.27 1.27)
+				)
+			)
+		)
+		(property "Datasheet" ""
+			(at 228.6 71.12 0)
+			(hide yes)
+			(show_name no)
+			(do_not_autoplace no)
+			(effects
+				(font
+					(size 1.27 1.27)
+				)
+			)
+		)
+		(property "Description" "Special symbol for telling ERC where power comes from"
+			(at 228.6 71.12 0)
+			(hide yes)
+			(show_name no)
+			(do_not_autoplace no)
+			(effects
+				(font
+					(size 1.27 1.27)
+				)
+			)
+		)
+		(pin "1"
+		)
+		(instances
+			(project "stm32f303-module"
+				(path "/1ffc8a7d-446d-4d87-80cb-e72e4474d330"
+					(reference "#FLG01")
+					(unit 1)
+				)
+			)
+		)
+	)
+	(symbol
 		(lib_id "power:GND")
 		(at 251.46 68.58 0)
@@
 					(unit 1)
 				)
+			)
+		)
+	)
+	(symbol
+		(lib_id "power:PWR_FLAG")
+		(at 251.46 66.04 270)
+		(unit 1)
+		(body_style 1)
+		(exclude_from_sim no)
+		(in_bom yes)
+		(on_board yes)
+		(in_pos_files yes)
+		(dnp no)
+		(fields_autoplaced yes)
+		(property "Reference" "#FLG02"
+			(at 253.365 66.04 0)
+			(hide yes)
+			(show_name no)
+			(do_not_autoplace no)
+			(effects
+				(font
+					(size 1.27 1.27)
+				)
+			)
+		)
+		(property "Value" "PWR_FLAG"
+			(at 255.27 66.0399 90)
+			(show_name no)
+			(do_not_autoplace no)
+			(effects
+				(font
+					(size 1.27 1.27)
+				)
+				(justify left)
+			)
+		)
+		(property "Footprint" ""
+			(at 251.46 66.04 0)
+			(hide yes)
+			(show_name no)
+			(do_not_autoplace no)
+			(effects
+				(font
+					(size 1.27 1.27)
+				)
+			)
+		)
+		(property "Datasheet" ""
+			(at 251.46 66.04 0)
+			(hide yes)
+			(show_name no)
+			(do_not_autoplace no)
+			(effects
+				(font
+					(size 1.27 1.27)
+				)
+			)
+		)
+		(property "Description" "Special symbol for telling ERC where power comes from"
+			(at 251.46 66.04 0)
+			(hide yes)
+			(show_name no)
+			(do_not_autoplace no)
+			(effects
+				(font
+					(size 1.27 1.27)
+				)
+			)
+		)
+		(pin "1"
+		)
+		(instances
+			(project "stm32f303-module"
+				(path "/1ffc8a7d-446d-4d87-80cb-e72e4474d330"
+					(reference "#FLG02")
+					(unit 1)
+				)
